File: PCB/KiCAD/BPF_PA.sch (KiCad schematic (older format))
At the start: 36 parts, among them J4 Conn_Coaxial, J5 Conn_Coaxial, J7 Conn_Coaxial, K1 TQ2-12VDC, Q11 BFG591, Q12 IRF610, Q5 MMBT2222A, T1 1_9, T3 1_4

Commit message: diode mixer on discrete components, begin move to DragonFly libs
Parts:
- Q11: footprint TO_SOT_Packages_SMD:SOT-223 -> DragonFly:SOT-223
- Q5: footprint TO_SOT_Packages_SMD:SOT-23 -> DragonFly:SOT-23
Changed lines of the file:
@@
 EESchema Schematic File Version 2
 LIBS:DragonFly-rescue
-LIBS:bee-rescue
 LIBS:power
 LIBS:device
@@
 $EndComp
 $Comp
-L GND #PWR86
+L GND #PWR090
 U 1 1 60FCFCEB
 P 2600 3800
-F 0 "#PWR86" H 2600 3550 50  0001 C CNN
+F 0 "#PWR090" H 2600 3550 50  0001 C CNN
 F 1 "GND" H 2600 3650 50  0001 C CNN
 F 2 "" H 2600 3800 50  0001 C CNN
@@
 F 0 "Q11" H 5300 3300 50  0000 L CNN
 F 1 "BFG591" H 5300 3200 50  0000 L CNN
-F 2 "TO_SOT_Packages_SMD:SOT-223" H 5300 3350 50  0001 C CNN
+F 2 "DragonFly:SOT-223" H 5300 3350 50  0001 C CNN
 F 3 "" H 5100 3250 50  0001 C CNN
 	1    5100 3250
@@
 $EndComp
 $Comp
-L GND #PWR89
+L GND #PWR091
 U 1 1 60FD0762
 P 3900 3600
-F 0 "#PWR89" H 3900 3350 50  0001 C CNN
+F 0 "#PWR091" H 3900 3350 50  0001 C CNN
 F 1 "GND" H 3900 3450 50  0001 C CNN
 F 2 "" H 3900 3600 50  0001 C CNN
@@
 $EndComp
 $Comp
-L GND #PWR91
+L GND #PWR092
 U 1 1 60FD078E
 P 5150 3900
-F 0 "#PWR91" H 5150 3650 50  0001 C CNN
+F 0 "#PWR092" H 5150 3650 50  0001 C CNN
 F 1 "GND" H 5150 3750 50  0001 C CNN
 F 2 "" H 5150 3900 50  0001 C CNN
@@
 $EndComp
 $Comp
-L GND #PWR93
+L GND #PWR093
 U 1 1 60FD07BA
 P 5350 3900
-F 0 "#PWR93" H 5350 3650 50  0001 C CNN
+F 0 "#PWR093" H 5350 3650 50  0001 C CNN
 F 1 "GND" H 5350 3750 50  0001 C CNN
 F 2 "" H 5350 3900 50  0001 C CNN
@@
 $EndComp
 $Comp
-L GND #PWR92
+L GND #PWR094
 U 1 1 60FD37CB
 P 5200 2250
-F 0 "#PWR92" H 5200 2000 50  0001 C CNN
+F 0 "#PWR094" H 5200 2000 50  0001 C CNN
 F 1 "GND" H 5200 2100 50  0001 C CNN
 F 2 "" H 5200 2250 50  0001 C CNN
@@
 $EndComp
 $Comp
-L GND #PWR90
+L GND #PWR095
 U 1 1 60FD3870
 P 4600 2250
-F 0 "#PWR90" H 4600 2000 50  0001 C CNN
+F 0 "#PWR095" H 4600 2000 50  0001 C CNN
 F 1 "GND" H 4600 2100 50  0001 C CNN
 F 2 "" H 4600 2250 50  0001 C CNN
@@
 $EndComp
 $Comp
-L GND #PWR105
+L GND #PWR096
 U 1 1 60FD3B07
 P 7350 3500
-F 0 "#PWR105" H 7350 3250 50  0001 C CNN
+F 0 "#PWR096" H 7350 3250 50  0001 C CNN
 F 1 "GND" H 7350 3350 50  0001 C CNN
 F 2 "" H 7350 3500 50  0001 C CNN
@@
 $EndComp
 $Comp
-L GND #PWR96
+L GND #PWR097
 U 1 1 60FD4018
 P 6050 3950
-F 0 "#PWR96" H 6050 3700 50  0001 C CNN
+F 0 "#PWR097" H 6050 3700 50  0001 C CNN
 F 1 "GND" H 6050 3800 50  0001 C CNN
 F 2 "" H 6050 3950 50  0001 C CNN
@@
 $EndComp
 $Comp
-L GND #PWR100
+L GND #PWR098
 U 1 1 60FD41CF
 P 6900 3650
-F 0 "#PWR100" H 6900 3400 50  0001 C CNN
+F 0 "#PWR098" H 6900 3400 50  0001 C CNN
 F 1 "GND" H 6900 3500 50  0001 C CNN
 F 2 "" H 6900 3650 50  0001 C CNN
@@
 $EndComp
 $Comp
-L GND #PWR102
+L GND #PWR099
 U 1 1 60FD63D0
 P 6950 2550
-F 0 "#PWR102" H 6950 2300 50  0001 C CNN
+F 0 "#PWR099" H 6950 2300 50  0001 C CNN
 F 1 "GND" H 6950 2400 50  0001 C CNN
 F 2 "" H 6950 2550 50  0001 C CNN
@@
 $EndComp
 $Comp
-L GND #PWR101
+L GND #PWR0100
 U 1 1 60FD6513
 P 6950 2200
-F 0 "#PWR101" H 6950 1950 50  0001 C CNN
+F 0 "#PWR0100" H 6950 1950 50  0001 C CNN
 F 1 "GND" H 6950 2050 50  0001 C CNN
 F 2 "" H 6950 2200 50  0001 C CNN
@@
 $EndComp
 $Comp
-L GND #PWR98
+L GND #PWR0101
 U 1 1 60FD7124
 P 6850 4050
-F 0 "#PWR98" H 6850 3800 50  0001 C CNN
+F 0 "#PWR0101" H 6850 3800 50  0001 C CNN
 F 1 "GND" H 6850 3900 50  0001 C CNN
 F 2 "" H 6850 4050 50  0001 C CNN
@@
 $EndComp
 $Comp
-L GND #PWR99
+L GND #PWR0102
 U 1 1 60FD7200
 P 6850 4450
-F 0 "#PWR99" H 6850 4200 50  0001 C CNN
+F 0 "#PWR0102" H 6850 4200 50  0001 C CNN
 F 1 "GND" H 6850 4300 50  0001 C CNN
 F 2 "" H 6850 4450 50  0001 C CNN
@@
 $EndComp
 $Comp
-L +12V #PWR88
+L +12V #PWR0103
 U 1 1 60FD8C5E
 P 3650 1800
-F 0 "#PWR88" H 3650 1650 50  0001 C CNN
+F 0 "#PWR0103" H 3650 1650 50  0001 C CNN
 F 1 "+12V" V 3650 2050 50  0000 C CNN
 F 2 "" H 3650 1800 50  0001 C CNN
@@
 $EndComp
 $Comp
-L +12V #PWR104
+L +12V #PWR0104
 U 1 1 60FD8D87
 P 7350 1650
-F 0 "#PWR104" H 7350 1500 50  0001 C CNN
+F 0 "#PWR0104" H 7350 1500 50  0001 C CNN
 F 1 "+12V" H 7350 1790 50  0000 C CNN
 F 2 "" H 7350 1650 50  0001 C CNN
@@
 $EndComp
 $Comp
-L GND #PWR84
+L GND #PWR0105
 U 1 1 60FDD885
 P 2050 4400
-F 0 "#PWR84" H 2050 4150 50  0001 C CNN
+F 0 "#PWR0105" H 2050 4150 50  0001 C CNN
 F 1 "GND" H 2050 4250 50  0001 C CNN
 F 2 "" H 2050 4400 50  0001 C CNN
@@
 $EndComp
 $Comp
-L GND #PWR87
+L GND #PWR0106
 U 1 1 60FDD9BB
 P 3250 4400
-F 0 "#PWR87" H 3250 4150 50  0001 C CNN
+F 0 "#PWR0106" H 3250 4150 50  0001 C CNN
 F 1 "GND" H 3250 4250 50  0001 C CNN
 F 2 "" H 3250 4400 50  0001 C CNN
@@
 $EndComp
 $Comp
-L GND #PWR103
+L GND #PWR0107
 U 1 1 60FE3B69
 P 7300 6250
-F 0 "#PWR103" H 7300 6000 50  0001 C CNN
+F 0 "#PWR0107" H 7300 6000 50  0001 C CNN
 F 1 "GND" H 7300 6100 50  0001 C CNN
 F 2 "" H 7300 6250 50  0001 C CNN
@@
 $EndComp
 $Comp
-L GND #PWR95
+L GND #PWR0108
 U 1 1 6105582E
 P 5900 6300
-F 0 "#PWR95" H 5900 6050 50  0001 C CNN
+F 0 "#PWR0108" H 5900 6050 50  0001 C CNN
 F 1 "GND" H 5900 6150 50  0001 C CNN
 F 2 "" H 5900 6300 50  0001 C CNN
@@
 $EndComp
 $Comp
-L GND #PWR94
+L GND #PWR0109
 U 1 1 61055A33
 P 5500 6300
-F 0 "#PWR94" H 5500 6050 50  0001 C CNN
+F 0 "#PWR0109" H 5500 6050 50  0001 C CNN
 F 1 "GND" H 5500 6150 50  0001 C CNN
 F 2 "" H 5500 6300 50  0001 C CNN
@@
 $EndComp
 $Comp
-L GND #PWR97
+L GND #PWR0110
 U 1 1 61055FE5
 P 6750 6550
-F 0 "#PWR97" H 6750 6300 50  0001 C CNN
+F 0 "#PWR0110" H 6750 6300 50  0001 C CNN
 F 1 "GND" H 6750 6400 50  0001 C CNN
 F 2 "" H 6750 6550 50  0001 C CNN
@@
 F 0 "Q5" H 2550 6200 50  0000 L CNN
 F 1 "MMBT2222A" H 2550 6100 50  0000 L CNN
-F 2 "TO_SOT_Packages_SMD:SOT-23" H 2550 6250 50  0001 C CNN
+F 2 "DragonFly:SOT-23" H 2550 6250 50  0001 C CNN
 F 3 "" H 2350 6150 50  0001 C CNN
 	1    2350 6150
@@
 $EndComp
 $Comp
-L GND #PWR85
+L GND #PWR0111
 U 1 1 61056E24
 P 2450 6400
-F 0 "#PWR85" H 2450 6150 50  0001 C CNN
+F 0 "#PWR0111" H 2450 6150 50  0001 C CNN
 F 1 "GND" H 2450 6250 50  0001 C CNN
 F 2 "" H 2450 6400 50  0001 C CNN

Commit message: begin BPF
Parts:
- added C61, C64: 560pF, DragonFly:C_1206_0603, symbol C_Small
- added C62, C63: C_Variable, Capacitors_SMD:C_Trimmer_Voltronics_JZ, symbol C_Variable
- C44: value 390pF -> 1nF
- J4, J5: footprint (none) -> DragonFly:U.FL_Molex_MCRF_73412-0110_Vertical
- L6, L7: value 52uH -> 31uH; footprint (none) -> DragonFly:Choke_Toroid_5x10mm_Vertical
- Q12: footprint TO_SOT_Packages_THT:TO-220-3_Horizontal -> DragonFly:TO-220_Neutral123_Horizontal_LargePads
Connections:
- wire segments 103 -> 113
Other:
- moved on the sheet: C43, C44, C45, C46, C47, C48, C49, C50, C51, C52, C53, E1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

Commit message: PCB read works, layout BPF
Parts:
- removed Q12: IRF610, DragonFly:TO-220_Neutral123_Horizontal_LargePads, symbol IRF540N
- added C65: 10nF, DragonFly:C_0603_HandSoldering, symbol C_Small
- added C66, C67: 560pF, DragonFly:C_1206_0603, symbol C_Small
- added D11: LL4148, DragonFly:MiniMELF_Standard, symbol D_Small
- added L5: 1uH, DragonFly:Choke_Toroid_5x10mm_Vertical, symbol L_Small
- added Q7: IRF610, DragonFly:TO-220_Neutral123_Horizontal_LargePads, symbol Q_NMOS_GDS
- added R38: 3.3K, DragonFly:R_1206_0603, symbol R_Small
- C47: footprint Capacitors_THT:CP_Radial_D4.0mm_P2.00mm -> DragonFly:CP_Radial_D4.0mm_P2.00mm
- C48, C53: footprint Capacitors_SMD:C_0603_HandSoldering -> DragonFly:C_0603_HandSoldering
- J7: value Conn_Coaxial -> ANT; footprint Connectors:SMA_THT_Jack_Straight -> DragonFly:SMA_THT_Jack_Straight
- R20: footprint (none) -> DragonFly:C_0603_HandSoldering
- R28: footprint (none) -> DragonFly:R_0603_HandSoldering
- R29, R30, R31: footprint (none) -> DragonFly:R_1206_0603
- T1: footprint (none) -> DragonFly:HF12
Connections:
- net labels added: TX_PA
- wire segments 113 -> 127
Other:
- note added: "Band Pass Filter Zin=Zout=50R 7Mhz\n"
- moved on the sheet: E1, J7, Q5

Commit message: PCB progress, QER filter place, PA place
Connections:
- net at Q11.2 (B), R22.2, R24.2: now also C53.2; no longer R31.2
- net at Q11.4 (C), T1.1: now also R31.2; no longer C53.2
Other:
- moved on the sheet: C53
Changed lines of the file:
@@
 $EndComp
 $Comp
-L GND #PWR090
+L GND #PWR93
 U 1 1 60FCFCEB
 P 3100 2900
-F 0 "#PWR090" H 3100 2650 50  0001 C CNN
+F 0 "#PWR93" H 3100 2650 50  0001 C CNN
 F 1 "GND" H 3100 2750 50  0001 C CNN
 F 2 "" H 3100 2900 50  0001 C CNN
@@
 $EndComp
 $Comp
-L GND #PWR091
+L GND #PWR98
 U 1 1 60FD0762
 P 5250 2800
-F 0 "#PWR091" H 5250 2550 50  0001 C CNN
+F 0 "#PWR98" H 5250 2550 50  0001 C CNN
 F 1 "GND" H 5250 2650 50  0001 C CNN
 F 2 "" H 5250 2800 50  0001 C CNN
@@
 $EndComp
 $Comp
-L GND #PWR092
+L GND #PWR102
 U 1 1 60FD078E
 P 6500 3100
-F 0 "#PWR092" H 6500 2850 50  0001 C CNN
+F 0 "#PWR102" H 6500 2850 50  0001 C CNN
 F 1 "GND" H 6500 2950 50  0001 C CNN
 F 2 "" H 6500 3100 50  0001 C CNN
@@
 $EndComp
 $Comp
-L GND #PWR093
+L GND #PWR105
 U 1 1 60FD07BA
 P 6700 3100
-F 0 "#PWR093" H 6700 2850 50  0001 C CNN
+F 0 "#PWR105" H 6700 2850 50  0001 C CNN
 F 1 "GND" H 6700 2950 50  0001 C CNN
 F 2 "" H 6700 3100 50  0001 C CNN
@@
 $EndComp
 $Comp
-L GND #PWR094
+L GND #PWR103
 U 1 1 60FD37CB
 P 6550 1450
-F 0 "#PWR094" H 6550 1200 50  0001 C CNN
+F 0 "#PWR103" H 6550 1200 50  0001 C CNN
 F 1 "GND" H 6550 1300 50  0001 C CNN
 F 2 "" H 6550 1450 50  0001 C CNN
@@
 $EndComp
 $Comp
-L GND #PWR095
+L GND #PWR101
 U 1 1 60FD3870
 P 5950 1450
-F 0 "#PWR095" H 5950 1200 50  0001 C CNN
+F 0 "#PWR101" H 5950 1200 50  0001 C CNN
 F 1 "GND" H 5950 1300 50  0001 C CNN
 F 2 "" H 5950 1450 50  0001 C CNN
@@
 $EndComp
 $Comp
-L GND #PWR096
+L GND #PWR116
 U 1 1 60FD3B07
 P 8700 2700
-F 0 "#PWR096" H 8700 2450 50  0001 C CNN
+F 0 "#PWR116" H 8700 2450 50  0001 C CNN
 F 1 "GND" H 8700 2550 50  0001 C CNN
 F 2 "" H 8700 2700 50  0001 C CNN
@@
 $EndComp
 $Comp
-L GND #PWR097
+L GND #PWR107
 U 1 1 60FD4018
 P 7400 3150
-F 0 "#PWR097" H 7400 2900 50  0001 C CNN
+F 0 "#PWR107" H 7400 2900 50  0001 C CNN
 F 1 "GND" H 7400 3000 50  0001 C CNN
 F 2 "" H 7400 3150 50  0001 C CNN
@@
 $EndComp
 $Comp
-L GND #PWR098
+L GND #PWR112
 U 1 1 60FD41CF
 P 8250 2850
-F 0 "#PWR098" H 8250 2600 50  0001 C CNN
+F 0 "#PWR112" H 8250 2600 50  0001 C CNN
 F 1 "GND" H 8250 2700 50  0001 C CNN
 F 2 "" H 8250 2850 50  0001 C CNN
@@
 $EndComp
 $Comp
-L GND #PWR099
+L GND #PWR114
 U 1 1 60FD63D0
 P 8300 1750
-F 0 "#PWR099" H 8300 1500 50  0001 C CNN
+F 0 "#PWR114" H 8300 1500 50  0001 C CNN
 F 1 "GND" H 8300 1600 50  0001 C CNN
 F 2 "" H 8300 1750 50  0001 C CNN
@@
 $EndComp
 $Comp
-L GND #PWR0100
+L GND #PWR113
 U 1 1 60FD6513
 P 8300 1400
-F 0 "#PWR0100" H 8300 1150 50  0001 C CNN
+F 0 "#PWR113" H 8300 1150 50  0001 C CNN
 F 1 "GND" H 8300 1250 50  0001 C CNN
 F 2 "" H 8300 1400 50  0001 C CNN
@@
 $EndComp
 $Comp
-L GND #PWR0101
+L GND #PWR110
 U 1 1 60FD7124
 P 8200 3250
-F 0 "#PWR0101" H 8200 3000 50  0001 C CNN
+F 0 "#PWR110" H 8200 3000 50  0001 C CNN
 F 1 "GND" H 8200 3100 50  0001 C CNN
 F 2 "" H 8200 3250 50  0001 C CNN
@@
 $EndComp
 $Comp
-L GND #PWR0102
+L GND #PWR111
 U 1 1 60FD7200
 P 8200 3650
-F 0 "#PWR0102" H 8200 3400 50  0001 C CNN
+F 0 "#PWR111" H 8200 3400 50  0001 C CNN
 F 1 "GND" H 8200 3500 50  0001 C CNN
 F 2 "" H 8200 3650 50  0001 C CNN
@@
 $EndComp
 $Comp
-L +12V #PWR0103
+L +12V #PWR97
 U 1 1 60FD8C5E
 P 5000 1000
-F 0 "#PWR0103" H 5000 850 50  0001 C CNN
+F 0 "#PWR97" H 5000 850 50  0001 C CNN
 F 1 "+12V" V 5000 1250 50  0000 C CNN
 F 2 "" H 5000 1000 50  0001 C CNN
@@
 $EndComp
 $Comp
-L +12V #PWR0104
+L +12V #PWR115
 U 1 1 60FD8D87
 P 8700 850
-F 0 "#PWR0104" H 8700 700 50  0001 C CNN
+F 0 "#PWR115" H 8700 700 50  0001 C CNN
 F 1 "+12V" H 8700 990 50  0000 C CNN
 F 2 "" H 8700 850 50  0001 C CNN
@@
 $EndComp
 $Comp
-L GND #PWR0105
+L GND #PWR92
 U 1 1 60FDD885
 P 1750 3600
-F 0 "#PWR0105" H 1750 3350 50  0001 C CNN
+F 0 "#PWR92" H 1750 3350 50  0001 C CNN
 F 1 "GND" H 1750 3450 50  0001 C CNN
 F 2 "" H 1750 3600 50  0001 C CNN
@@
 $EndComp
 $Comp
-L GND #PWR0106
+L GND #PWR95
 U 1 1 60FDD9BB
 P 4600 3600
-F 0 "#PWR0106" H 4600 3350 50  0001 C CNN
+F 0 "#PWR95" H 4600 3350 50  0001 C CNN
 F 1 "GND" H 4600 3450 50  0001 C CNN
 F 2 "" H 4600 3600 50  0001 C CNN
@@
 $EndComp
 $Comp
-L GND #PWR0107
+L GND #PWR118
 U 1 1 60FE3B69
 P 9450 5450
-F 0 "#PWR0107" H 9450 5200 50  0001 C CNN
+F 0 "#PWR118" H 9450 5200 50  0001 C CNN
 F 1 "GND" H 9450 5300 50  0001 C CNN
 F 2 "" H 9450 5450 50  0001 C CNN
@@
 $EndComp
 $Comp
-L GND #PWR0108
+L GND #PWR109
 U 1 1 6105582E
 P 8050 5500
-F 0 "#PWR0108" H 8050 5250 50  0001 C CNN
+F 0 "#PWR109" H 8050 5250 50  0001 C CNN
 F 1 "GND" H 8050 5350 50  0001 C CNN
 F 2 "" H 8050 5500 50  0001 C CNN
@@
 $EndComp
 $Comp
-L GND #PWR0109
+L GND #PWR108
 U 1 1 61055A33
 P 7650 5500
-F 0 "#PWR0109" H 7650 5250 50  0001 C CNN
+F 0 "#PWR108" H 7650 5250 50  0001 C CNN
 F 1 "GND" H 7650 5350 50  0001 C CNN
 F 2 "" H 7650 5500 50  0001 C CNN
@@
 $EndComp
 $Comp
-L GND #PWR0110
+L GND #PWR117
 U 1 1 61055FE5
 P 8900 5750
-F 0 "#PWR0110" H 8900 5500 50  0001 C CNN
+F 0 "#PWR117" H 8900 5500 50  0001 C CNN
 F 1 "GND" H 8900 5600 50  0001 C CNN
 F 2 "" H 8900 5750 50  0001 C CNN
@@
 $EndComp
 $Comp
-L GND #PWR0111
+L GND #PWR100
 U 1 1 61056E24
 P 5850 5750
-F 0 "#PWR0111" H 5850 5500 50  0001 C CNN
+F 0 "#PWR100" H 5850 5500 50  0001 C CNN
 F 1 "GND" H 5850 5600 50  0001 C CNN
 F 2 "" H 5850 5750 50  0001 C CNN
@@
 $EndComp
 $Comp
-L R_Small R31
-U 1 1 6105F33F
+L C_Small C53
+U 1 1 610601CA
 P 5900 2300
-F 0 "R31" H 5950 2350 50  0000 L CNN
-F 1 "300R" H 5950 2250 50  0000 L CNN
-F 2 "DragonFly:R_1206_0603" H 5900 2300 50  0001 C CNN
+F 0 "C53" V 6100 2250 50  0000 L CNN
+F 1 "100nF" V 6000 2150 50  0000 L CNN
+F 2 "DragonFly:C_0603_HandSoldering" H 5900 2300 50  0001 C CNN
 F 3 "" H 5900 2300 50  0001 C CNN
 	1    5900 2300
 	1    0    0    -1
-$EndComp
-$Comp
-L C_Small C53
-U 1 1 610601CA
-P 6250 2100
-F 0 "C53" V 6450 2050 50  0000 L CNN
-F 1 "100nF" V 6350 1950 50  0000 L CNN
-F 2 "DragonFly:C_0603_HandSoldering" H 6250 2100 50  0001 C CNN
-F 3 "" H 6250 2100 50  0001 C CNN
-	1    6250 2100
-	0    -1   -1   0
 $EndComp
 Wire Wire Line
@@
 $EndComp
 $Comp
-L GND #PWR0112
+L GND #PWR91
 U 1 1 612355AA
 P 1750 2900
-F 0 "#PWR0112" H 1750 2650 50  0001 C CNN
+F 0 "#PWR91" H 1750 2650 50  0001 C CNN
 F 1 "GND" H 1750 2750 50  0001 C CNN
 F 2 "" H 1750 2900 50  0001 C CNN
@@
 $EndComp
 $Comp
-L GND #PWR0113
+L GND #PWR94
 U 1 1 612356A3
 P 4400 2900
-F 0 "#PWR0113" H 4400 2650 50  0001 C CNN
+F 0 "#PWR94" H 4400 2650 50  0001 C CNN
 F 1 "GND" H 4400 2750 50  0001 C CNN
 F 2 "" H 4400 2900 50  0001 C CNN
@@
 Connection ~ 5300 5500
 $Comp
-L GND #PWR0114
+L GND #PWR99
 U 1 1 61244496
 P 5300 5750
-F 0 "#PWR0114" H 5300 5500 50  0001 C CNN
+F 0 "#PWR99" H 5300 5500 50  0001 C CNN
 F 1 "GND" H 5300 5600 50  0001 C CNN
 F 2 "" H 5300 5750 50  0001 C CNN
@@
 $EndComp
 $Comp
-L +12V #PWR0115
+L +12V #PWR96
 U 1 1 61244868
 P 4600 4850
-F 0 "#PWR0115" H 4600 4700 50  0001 C CNN
+F 0 "#PWR96" H 4600 4700 50  0001 C CNN
 F 1 "+12V" V 4600 5100 50  0000 C CNN
 F 2 "" H 4600 4850 50  0001 C CNN
@@
 Connection ~ 7200 5150
 $Comp
-L GND #PWR0116
+L GND #PWR106
 U 1 1 6124C7E1
 P 7200 5500
-F 0 "#PWR0116" H 7200 5250 50  0001 C CNN
+F 0 "#PWR106" H 7200 5250 50  0001 C CNN
 F 1 "GND" H 7200 5350 50  0001 C CNN
 F 2 "" H 7200 5500 50  0001 C CNN
@@
 	7200 5500 7200 5450
 $Comp
-L GND #PWR0117
+L GND #PWR104
 U 1 1 6124C940
 P 6650 5500
-F 0 "#PWR0117" H 6650 5250 50  0001 C CNN
+F 0 "#PWR104" H 6650 5250 50  0001 C CNN
 F 1 "GND" H 6650 5350 50  0001 C CNN
 F 2 "" H 6650 5500 50  0001 C CNN
@@
 	1    0    0    -1
 $EndComp
+$Comp
+L R_Small R31
+U 1 1 61265F9A
+P 6250 2100
+F 0 "R31" V 6450 2050 50  0000 L CNN
+F 1 "300R" V 6350 2000 50  0000 L CNN
+F 2 "DragonFly:R_1206_0603" H 6250 2100 50  0001 C CNN
+F 3 "" H 6250 2100 50  0001 C CNN
+	1    6250 2100
+	0    -1   -1   0
+$EndComp
 $EndSCHEMATC
