File: PCB/KiCAD/BPF_PA.sch (KiCad schematic (older format))
At the start: 48 parts, among them CON2 BARREL_JACK, J4 Conn_Coaxial, J5 Conn_Coaxial, J7 ANT, K1 TQ2-12VDC, Q11 BFG591, Q5 MMBT2222A, Q7 IRF610, T1 1_9, T3 1_4

Commit message: PCB v1.0
Parts:
- C46, C50, C52: footprint Capacitors_SMD:C_0603_HandSoldering -> DragonFly:C_1206_0603
- C53: footprint DragonFly:C_0603_HandSoldering -> DragonFly:C_1206_0603
- L8: footprint (none) -> DragonFly:Choke_CD54
- R20: footprint DragonFly:C_0603_HandSoldering -> DragonFly:R_1206_0603
- R28: footprint DragonFly:R_0603_HandSoldering -> DragonFly:R_1206_0603
Changed lines of the file:
@@
 $EndComp
 $Comp
-L GND #PWR98
+L GND #PWR101
 U 1 1 60FCFCEB
 P 3100 2900
-F 0 "#PWR98" H 3100 2650 50  0001 C CNN
+F 0 "#PWR101" H 3100 2650 50  0001 C CNN
 F 1 "GND" H 3100 2750 50  0001 C CNN
 F 2 "" H 3100 2900 50  0001 C CNN
@@
 F 0 "R20" H 5300 2700 50  0000 L CNN
 F 1 "1K" H 5300 2600 50  0000 L CNN
-F 2 "DragonFly:C_0603_HandSoldering" H 5250 2650 50  0001 C CNN
+F 2 "DragonFly:R_1206_0603" H 5250 2650 50  0001 C CNN
 F 3 "" H 5250 2650 50  0001 C CNN
 	1    5250 2650
@@
 $EndComp
 $Comp
-L GND #PWR103
+L GND #PWR106
 U 1 1 60FD0762
 P 5250 2800
-F 0 "#PWR103" H 5250 2550 50  0001 C CNN
+F 0 "#PWR106" H 5250 2550 50  0001 C CNN
 F 1 "GND" H 5250 2650 50  0001 C CNN
 F 2 "" H 5250 2800 50  0001 C CNN
@@
 $EndComp
 $Comp
-L GND #PWR107
+L GND #PWR110
 U 1 1 60FD078E
 P 6500 3100
-F 0 "#PWR107" H 6500 2850 50  0001 C CNN
+F 0 "#PWR110" H 6500 2850 50  0001 C CNN
 F 1 "GND" H 6500 2950 50  0001 C CNN
 F 2 "" H 6500 3100 50  0001 C CNN
@@
 $EndComp
 $Comp
-L GND #PWR110
+L GND #PWR113
 U 1 1 60FD07BA
 P 6700 3100
-F 0 "#PWR110" H 6700 2850 50  0001 C CNN
+F 0 "#PWR113" H 6700 2850 50  0001 C CNN
 F 1 "GND" H 6700 2950 50  0001 C CNN
 F 2 "" H 6700 3100 50  0001 C CNN
@@
 F 0 "C46" H 6050 1300 50  0000 L CNN
 F 1 "100nF" H 6050 1200 50  0000 L CNN
-F 2 "Capacitors_SMD:C_0603_HandSoldering" H 5950 1250 50  0001 C CNN
+F 2 "DragonFly:C_1206_0603" H 5950 1250 50  0001 C CNN
 F 3 "" H 5950 1250 50  0001 C CNN
 	1    5950 1250
@@
 $EndComp
 $Comp
-L GND #PWR108
+L GND #PWR111
 U 1 1 60FD37CB
 P 6550 1450
-F 0 "#PWR108" H 6550 1200 50  0001 C CNN
+F 0 "#PWR111" H 6550 1200 50  0001 C CNN
 F 1 "GND" H 6550 1300 50  0001 C CNN
 F 2 "" H 6550 1450 50  0001 C CNN
@@
 $EndComp
 $Comp
-L GND #PWR106
+L GND #PWR109
 U 1 1 60FD3870
 P 5950 1450
-F 0 "#PWR106" H 5950 1200 50  0001 C CNN
+F 0 "#PWR109" H 5950 1200 50  0001 C CNN
 F 1 "GND" H 5950 1300 50  0001 C CNN
 F 2 "" H 5950 1450 50  0001 C CNN
@@
 $EndComp
 $Comp
-L GND #PWR121
+L GND #PWR124
 U 1 1 60FD3B07
 P 8700 2700
-F 0 "#PWR121" H 8700 2450 50  0001 C CNN
+F 0 "#PWR124" H 8700 2450 50  0001 C CNN
 F 1 "GND" H 8700 2550 50  0001 C CNN
 F 2 "" H 8700 2700 50  0001 C CNN
@@
 $EndComp
 $Comp
-L GND #PWR112
+L GND #PWR115
 U 1 1 60FD4018
 P 7400 3150
-F 0 "#PWR112" H 7400 2900 50  0001 C CNN
+F 0 "#PWR115" H 7400 2900 50  0001 C CNN
 F 1 "GND" H 7400 3000 50  0001 C CNN
 F 2 "" H 7400 3150 50  0001 C CNN
@@
 F 0 "R28" H 8300 2750 50  0000 L CNN
 F 1 "10k" H 8300 2650 50  0000 L CNN
-F 2 "DragonFly:R_0603_HandSoldering" H 8250 2700 50  0001 C CNN
+F 2 "DragonFly:R_1206_0603" H 8250 2700 50  0001 C CNN
 F 3 "" H 8250 2700 50  0001 C CNN
 	1    8250 2700
@@
 $EndComp
 $Comp
-L GND #PWR117
+L GND #PWR120
 U 1 1 60FD41CF
 P 8250 2850
-F 0 "#PWR117" H 8250 2600 50  0001 C CNN
+F 0 "#PWR120" H 8250 2600 50  0001 C CNN
 F 1 "GND" H 8250 2700 50  0001 C CNN
 F 2 "" H 8250 2850 50  0001 C CNN
@@
 F 0 "C52" V 8650 1700 50  0000 L CNN
 F 1 "100nF" V 8550 1600 50  0000 L CNN
-F 2 "Capacitors_SMD:C_0603_HandSoldering" H 8450 1750 50  0001 C CNN
+F 2 "DragonFly:C_1206_0603" H 8450 1750 50  0001 C CNN
 F 3 "" H 8450 1750 50  0001 C CNN
 	1    8450 1750
@@
 F 0 "L8" H 8750 1300 50  0000 L CNN
 F 1 "4.7µH" H 8750 1200 50  0000 L CNN
-F 2 "" H 8700 1200 50  0001 C CNN
+F 2 "DragonFly:Choke_CD54" H 8700 1200 50  0001 C CNN
 F 3 "" H 8700 1200 50  0001 C CNN
 	1    8700 1200
@@
 $EndComp
 $Comp
-L GND #PWR119
+L GND #PWR122
 U 1 1 60FD63D0
 P 8300 1750
-F 0 "#PWR119" H 8300 1500 50  0001 C CNN
+F 0 "#PWR122" H 8300 1500 50  0001 C CNN
 F 1 "GND" H 8300 1600 50  0001 C CNN
 F 2 "" H 8300 1750 50  0001 C CNN
@@
 $EndComp
 $Comp
-L GND #PWR118
+L GND #PWR121
 U 1 1 60FD6513
 P 8300 1400
-F 0 "#PWR118" H 8300 1150 50  0001 C CNN
+F 0 "#PWR121" H 8300 1150 50  0001 C CNN
 F 1 "GND" H 8300 1250 50  0001 C CNN
 F 2 "" H 8300 1400 50  0001 C CNN
@@
 F 0 "C50" V 8200 3600 50  0000 L CNN
 F 1 "100nF" V 8100 3500 50  0000 L CNN
-F 2 "Capacitors_SMD:C_0603_HandSoldering" H 8000 3650 50  0001 C CNN
+F 2 "DragonFly:C_1206_0603" H 8000 3650 50  0001 C CNN
 F 3 "" H 8000 3650 50  0001 C CNN
 	1    8000 3650
@@
 $EndComp
 $Comp
-L GND #PWR115
+L GND #PWR118
 U 1 1 60FD7124
 P 8200 3250
-F 0 "#PWR115" H 8200 3000 50  0001 C CNN
+F 0 "#PWR118" H 8200 3000 50  0001 C CNN
 F 1 "GND" H 8200 3100 50  0001 C CNN
 F 2 "" H 8200 3250 50  0001 C CNN
@@
 $EndComp
 $Comp
-L GND #PWR116
+L GND #PWR119
 U 1 1 60FD7200
 P 8200 3650
-F 0 "#PWR116" H 8200 3400 50  0001 C CNN
+F 0 "#PWR119" H 8200 3400 50  0001 C CNN
 F 1 "GND" H 8200 3500 50  0001 C CNN
 F 2 "" H 8200 3650 50  0001 C CNN
@@
 $EndComp
 $Comp
-L +12V #PWR102
+L +12V #PWR105
 U 1 1 60FD8C5E
 P 5000 1000
-F 0 "#PWR102" H 5000 850 50  0001 C CNN
+F 0 "#PWR105" H 5000 850 50  0001 C CNN
 F 1 "+12V" V 5000 1250 50  0000 C CNN
 F 2 "" H 5000 1000 50  0001 C CNN
@@
 $EndComp
 $Comp
-L +12V #PWR120
+L +12V #PWR123
 U 1 1 60FD8D87
 P 8700 850
-F 0 "#PWR120" H 8700 700 50  0001 C CNN
+F 0 "#PWR123" H 8700 700 50  0001 C CNN
 F 1 "+12V" H 8700 990 50  0000 C CNN
 F 2 "" H 8700 850 50  0001 C CNN
@@
 $EndComp
 $Comp
-L GND #PWR95
+L GND #PWR98
 U 1 1 60FDD885
 P 1750 3600
-F 0 "#PWR95" H 1750 3350 50  0001 C CNN
+F 0 "#PWR98" H 1750 3350 50  0001 C CNN
 F 1 "GND" H 1750 3450 50  0001 C CNN
 F 2 "" H 1750 3600 50  0001 C CNN
@@
 $EndComp
 $Comp
-L GND #PWR100
+L GND #PWR103
 U 1 1 60FDD9BB
 P 4600 3600
-F 0 "#PWR100" H 4600 3350 50  0001 C CNN
+F 0 "#PWR103" H 4600 3350 50  0001 C CNN
 F 1 "GND" H 4600 3450 50  0001 C CNN
 F 2 "" H 4600 3600 50  0001 C CNN
@@
 $EndComp
 $Comp
-L GND #PWR123
+L GND #PWR126
 U 1 1 60FE3B69
 P 9450 5450
-F 0 "#PWR123" H 9450 5200 50  0001 C CNN
+F 0 "#PWR126" H 9450 5200 50  0001 C CNN
 F 1 "GND" H 9450 5300 50  0001 C CNN
 F 2 "" H 9450 5450 50  0001 C CNN
@@
 $EndComp
 $Comp
-L GND #PWR114
+L GND #PWR117
 U 1 1 6105582E
 P 8050 5500
-F 0 "#PWR114" H 8050 5250 50  0001 C CNN
+F 0 "#PWR117" H 8050 5250 50  0001 C CNN
 F 1 "GND" H 8050 5350 50  0001 C CNN
 F 2 "" H 8050 5500 50  0001 C CNN
@@
 $EndComp
 $Comp
-L GND #PWR113
+L GND #PWR116
 U 1 1 61055A33
 P 7650 5500
-F 0 "#PWR113" H 7650 5250 50  0001 C CNN
+F 0 "#PWR116" H 7650 5250 50  0001 C CNN
 F 1 "GND" H 7650 5350 50  0001 C CNN
 F 2 "" H 7650 5500 50  0001 C CNN
@@
 $EndComp
 $Comp
-L GND #PWR122
+L GND #PWR125
 U 1 1 61055FE5
 P 8900 5750
-F 0 "#PWR122" H 8900 5500 50  0001 C CNN
+F 0 "#PWR125" H 8900 5500 50  0001 C CNN
 F 1 "GND" H 8900 5600 50  0001 C CNN
 F 2 "" H 8900 5750 50  0001 C CNN
@@
 $EndComp
 $Comp
-L GND #PWR105
+L GND #PWR108
 U 1 1 61056E24
 P 5850 5750
-F 0 "#PWR105" H 5850 5500 50  0001 C CNN
+F 0 "#PWR108" H 5850 5500 50  0001 C CNN
 F 1 "GND" H 5850 5600 50  0001 C CNN
 F 2 "" H 5850 5750 50  0001 C CNN
@@
 U 1 1 610601CA
 P 5900 2300
-F 0 "C53" V 6100 2250 50  0000 L CNN
-F 1 "100nF" V 6000 2150 50  0000 L CNN
-F 2 "DragonFly:C_0603_HandSoldering" H 5900 2300 50  0001 C CNN
+F 0 "C53" H 6000 2400 50  0000 L CNN
+F 1 "100nF" H 6000 2300 50  0000 L CNN
+F 2 "DragonFly:C_1206_0603" H 5900 2300 50  0001 C CNN
 F 3 "" H 5900 2300 50  0001 C CNN
 	1    5900 2300
@@
 $EndComp
 $Comp
-L GND #PWR94
+L GND #PWR97
 U 1 1 612355AA
 P 1750 2900
-F 0 "#PWR94" H 1750 2650 50  0001 C CNN
+F 0 "#PWR97" H 1750 2650 50  0001 C CNN
 F 1 "GND" H 1750 2750 50  0001 C CNN
 F 2 "" H 1750 2900 50  0001 C CNN
@@
 $EndComp
 $Comp
-L GND #PWR99
+L GND #PWR102
 U 1 1 612356A3
 P 4400 2900
-F 0 "#PWR99" H 4400 2650 50  0001 C CNN
+F 0 "#PWR102" H 4400 2650 50  0001 C CNN
 F 1 "GND" H 4400 2750 50  0001 C CNN
 F 2 "" H 4400 2900 50  0001 C CNN
@@
 Connection ~ 5300 5500
 $Comp
-L GND #PWR104
+L GND #PWR107
 U 1 1 61244496
 P 5300 5750
-F 0 "#PWR104" H 5300 5500 50  0001 C CNN
+F 0 "#PWR107" H 5300 5500 50  0001 C CNN
 F 1 "GND" H 5300 5600 50  0001 C CNN
 F 2 "" H 5300 5750 50  0001 C CNN
@@
 $EndComp
 $Comp
-L +12V #PWR101
+L +12V #PWR104
 U 1 1 61244868
 P 4600 4850
-F 0 "#PWR101" H 4600 4700 50  0001 C CNN
+F 0 "#PWR104" H 4600 4700 50  0001 C CNN
 F 1 "+12V" V 4600 5100 50  0000 C CNN
 F 2 "" H 4600 4850 50  0001 C CNN
@@
 Connection ~ 7200 5150
 $Comp
-L GND #PWR111
+L GND #PWR114
 U 1 1 6124C7E1
 P 7200 5500
-F 0 "#PWR111" H 7200 5250 50  0001 C CNN
+F 0 "#PWR114" H 7200 5250 50  0001 C CNN
 F 1 "GND" H 7200 5350 50  0001 C CNN
 F 2 "" H 7200 5500 50  0001 C CNN
@@
 	7200 5500 7200 5450
 $Comp
-L GND #PWR109
+L GND #PWR112
 U 1 1 6124C940
 P 6650 5500
-F 0 "#PWR109" H 6650 5250 50  0001 C CNN
+F 0 "#PWR112" H 6650 5250 50  0001 C CNN
 F 1 "GND" H 6650 5350 50  0001 C CNN
 F 2 "" H 6650 5500 50  0001 C CNN
@@
 $EndComp
 $Comp
-L +12V #PWR97
+L +12V #PWR100
 U 1 1 6126FE6E
 P 2700 5250
-F 0 "#PWR97" H 2700 5100 50  0001 C CNN
+F 0 "#PWR100" H 2700 5100 50  0001 C CNN
 F 1 "+12V" V 2700 5500 50  0000 C CNN
 F 2 "" H 2700 5250 50  0001 C CNN
@@
 $EndComp
 $Comp
-L GND #PWR96
+L GND #PWR99
 U 1 1 612713A0
 P 2650 5850
-F 0 "#PWR96" H 2650 5600 50  0001 C CNN
+F 0 "#PWR99" H 2650 5600 50  0001 C CNN
 F 1 "GND" H 2650 5700 50  0001 C CNN
 F 2 "" H 2650 5850 50  0001 C CNN

Commit message: PCB production
Parts:
- E1: footprint (none) -> DragonFly:Resistor_Vertical_RM5mm
Changed lines of the file:
@@
 $EndComp
 $Comp
-L GND #PWR101
+L GND #PWR097
 U 1 1 60FCFCEB
 P 3100 2900
-F 0 "#PWR101" H 3100 2650 50  0001 C CNN
+F 0 "#PWR097" H 3100 2650 50  0001 C CNN
 F 1 "GND" H 3100 2750 50  0001 C CNN
 F 2 "" H 3100 2900 50  0001 C CNN
@@
 $EndComp
 $Comp
-L GND #PWR106
+L GND #PWR098
 U 1 1 60FD0762
 P 5250 2800
-F 0 "#PWR106" H 5250 2550 50  0001 C CNN
+F 0 "#PWR098" H 5250 2550 50  0001 C CNN
 F 1 "GND" H 5250 2650 50  0001 C CNN
 F 2 "" H 5250 2800 50  0001 C CNN
@@
 $EndComp
 $Comp
-L GND #PWR110
+L GND #PWR099
 U 1 1 60FD078E
 P 6500 3100
-F 0 "#PWR110" H 6500 2850 50  0001 C CNN
+F 0 "#PWR099" H 6500 2850 50  0001 C CNN
 F 1 "GND" H 6500 2950 50  0001 C CNN
 F 2 "" H 6500 3100 50  0001 C CNN
@@
 $EndComp
 $Comp
-L GND #PWR113
+L GND #PWR0100
 U 1 1 60FD07BA
 P 6700 3100
-F 0 "#PWR113" H 6700 2850 50  0001 C CNN
+F 0 "#PWR0100" H 6700 2850 50  0001 C CNN
 F 1 "GND" H 6700 2950 50  0001 C CNN
 F 2 "" H 6700 3100 50  0001 C CNN
@@
 $EndComp
 $Comp
-L GND #PWR111
+L GND #PWR0101
 U 1 1 60FD37CB
 P 6550 1450
-F 0 "#PWR111" H 6550 1200 50  0001 C CNN
+F 0 "#PWR0101" H 6550 1200 50  0001 C CNN
 F 1 "GND" H 6550 1300 50  0001 C CNN
 F 2 "" H 6550 1450 50  0001 C CNN
@@
 $EndComp
 $Comp
-L GND #PWR109
+L GND #PWR0102
 U 1 1 60FD3870
 P 5950 1450
-F 0 "#PWR109" H 5950 1200 50  0001 C CNN
+F 0 "#PWR0102" H 5950 1200 50  0001 C CNN
 F 1 "GND" H 5950 1300 50  0001 C CNN
 F 2 "" H 5950 1450 50  0001 C CNN
@@
 $EndComp
 $Comp
-L GND #PWR124
+L GND #PWR0103
 U 1 1 60FD3B07
 P 8700 2700
-F 0 "#PWR124" H 8700 2450 50  0001 C CNN
+F 0 "#PWR0103" H 8700 2450 50  0001 C CNN
 F 1 "GND" H 8700 2550 50  0001 C CNN
 F 2 "" H 8700 2700 50  0001 C CNN
@@
 $EndComp
 $Comp
-L GND #PWR115
+L GND #PWR0104
 U 1 1 60FD4018
 P 7400 3150
-F 0 "#PWR115" H 7400 2900 50  0001 C CNN
+F 0 "#PWR0104" H 7400 2900 50  0001 C CNN
 F 1 "GND" H 7400 3000 50  0001 C CNN
 F 2 "" H 7400 3150 50  0001 C CNN
@@
 $EndComp
 $Comp
-L GND #PWR120
+L GND #PWR0105
 U 1 1 60FD41CF
 P 8250 2850
-F 0 "#PWR120" H 8250 2600 50  0001 C CNN
+F 0 "#PWR0105" H 8250 2600 50  0001 C CNN
 F 1 "GND" H 8250 2700 50  0001 C CNN
 F 2 "" H 8250 2850 50  0001 C CNN
@@
 $EndComp
 $Comp
-L GND #PWR122
+L GND #PWR0106
 U 1 1 60FD63D0
 P 8300 1750
-F 0 "#PWR122" H 8300 1500 50  0001 C CNN
+F 0 "#PWR0106" H 8300 1500 50  0001 C CNN
 F 1 "GND" H 8300 1600 50  0001 C CNN
 F 2 "" H 8300 1750 50  0001 C CNN
@@
 $EndComp
 $Comp
-L GND #PWR121
+L GND #PWR0107
 U 1 1 60FD6513
 P 8300 1400
-F 0 "#PWR121" H 8300 1150 50  0001 C CNN
+F 0 "#PWR0107" H 8300 1150 50  0001 C CNN
 F 1 "GND" H 8300 1250 50  0001 C CNN
 F 2 "" H 8300 1400 50  0001 C CNN
@@
 $EndComp
 $Comp
-L GND #PWR118
+L GND #PWR0108
 U 1 1 60FD7124
 P 8200 3250
-F 0 "#PWR118" H 8200 3000 50  0001 C CNN
+F 0 "#PWR0108" H 8200 3000 50  0001 C CNN
 F 1 "GND" H 8200 3100 50  0001 C CNN
 F 2 "" H 8200 3250 50  0001 C CNN
@@
 $EndComp
 $Comp
-L GND #PWR119
+L GND #PWR0109
 U 1 1 60FD7200
 P 8200 3650
-F 0 "#PWR119" H 8200 3400 50  0001 C CNN
+F 0 "#PWR0109" H 8200 3400 50  0001 C CNN
 F 1 "GND" H 8200 3500 50  0001 C CNN
 F 2 "" H 8200 3650 50  0001 C CNN
@@
 $EndComp
 $Comp
-L +12V #PWR105
+L +12V #PWR0110
 U 1 1 60FD8C5E
 P 5000 1000
-F 0 "#PWR105" H 5000 850 50  0001 C CNN
+F 0 "#PWR0110" H 5000 850 50  0001 C CNN
 F 1 "+12V" V 5000 1250 50  0000 C CNN
 F 2 "" H 5000 1000 50  0001 C CNN
@@
 $EndComp
 $Comp
-L +12V #PWR123
+L +12V #PWR0111
 U 1 1 60FD8D87
 P 8700 850
-F 0 "#PWR123" H 8700 700 50  0001 C CNN
+F 0 "#PWR0111" H 8700 700 50  0001 C CNN
 F 1 "+12V" H 8700 990 50  0000 C CNN
 F 2 "" H 8700 850 50  0001 C CNN
@@
 $EndComp
 $Comp
-L GND #PWR98
+L GND #PWR0112
 U 1 1 60FDD885
 P 1750 3600
-F 0 "#PWR98" H 1750 3350 50  0001 C CNN
+F 0 "#PWR0112" H 1750 3350 50  0001 C CNN
 F 1 "GND" H 1750 3450 50  0001 C CNN
 F 2 "" H 1750 3600 50  0001 C CNN
@@
 $EndComp
 $Comp
-L GND #PWR103
+L GND #PWR0113
 U 1 1 60FDD9BB
 P 4600 3600
-F 0 "#PWR103" H 4600 3350 50  0001 C CNN
+F 0 "#PWR0113" H 4600 3350 50  0001 C CNN
 F 1 "GND" H 4600 3450 50  0001 C CNN
 F 2 "" H 4600 3600 50  0001 C CNN
@@
 $EndComp
 $Comp
-L GND #PWR126
+L GND #PWR0114
 U 1 1 60FE3B69
 P 9450 5450
-F 0 "#PWR126" H 9450 5200 50  0001 C CNN
+F 0 "#PWR0114" H 9450 5200 50  0001 C CNN
 F 1 "GND" H 9450 5300 50  0001 C CNN
 F 2 "" H 9450 5450 50  0001 C CNN
@@
 $EndComp
 $Comp
-L GND #PWR117
+L GND #PWR0115
 U 1 1 6105582E
 P 8050 5500
-F 0 "#PWR117" H 8050 5250 50  0001 C CNN
+F 0 "#PWR0115" H 8050 5250 50  0001 C CNN
 F 1 "GND" H 8050 5350 50  0001 C CNN
 F 2 "" H 8050 5500 50  0001 C CNN
@@
 $EndComp
 $Comp
-L GND #PWR116
+L GND #PWR0116
 U 1 1 61055A33
 P 7650 5500
-F 0 "#PWR116" H 7650 5250 50  0001 C CNN
+F 0 "#PWR0116" H 7650 5250 50  0001 C CNN
 F 1 "GND" H 7650 5350 50  0001 C CNN
 F 2 "" H 7650 5500 50  0001 C CNN
@@
 F 0 "E1" V 8700 5150 50  0000 C CNN
 F 1 "SPARK_GAP" V 8800 5150 50  0000 C CNN
-F 2 "" H 8900 5380 50  0001 C CNN
+F 2 "DragonFly:Resistor_Vertical_RM5mm" H 8900 5380 50  0001 C CNN
 F 3 "" V 8900 5450 50  0001 C CNN
 	1    8900 5450
@@
 $EndComp
 $Comp
-L GND #PWR125
+L GND #PWR0117
 U 1 1 61055FE5
 P 8900 5750
-F 0 "#PWR125" H 8900 5500 50  0001 C CNN
+F 0 "#PWR0117" H 8900 5500 50  0001 C CNN
 F 1 "GND" H 8900 5600 50  0001 C CNN
 F 2 "" H 8900 5750 50  0001 C CNN
@@
 $EndComp
 $Comp
-L GND #PWR108
+L GND #PWR0118
 U 1 1 61056E24
 P 5850 5750
-F 0 "#PWR108" H 5850 5500 50  0001 C CNN
+F 0 "#PWR0118" H 5850 5500 50  0001 C CNN
 F 1 "GND" H 5850 5600 50  0001 C CNN
 F 2 "" H 5850 5750 50  0001 C CNN
@@
 $EndComp
 $Comp
-L GND #PWR97
+L GND #PWR0119
 U 1 1 612355AA
 P 1750 2900
-F 0 "#PWR97" H 1750 2650 50  0001 C CNN
+F 0 "#PWR0119" H 1750 2650 50  0001 C CNN
 F 1 "GND" H 1750 2750 50  0001 C CNN
 F 2 "" H 1750 2900 50  0001 C CNN
@@
 $EndComp
 $Comp
-L GND #PWR102
+L GND #PWR0120
 U 1 1 612356A3
 P 4400 2900
-F 0 "#PWR102" H 4400 2650 50  0001 C CNN
+F 0 "#PWR0120" H 4400 2650 50  0001 C CNN
 F 1 "GND" H 4400 2750 50  0001 C CNN
 F 2 "" H 4400 2900 50  0001 C CNN
@@
 Connection ~ 5300 5500
 $Comp
-L GND #PWR107
+L GND #PWR0121
 U 1 1 61244496
 P 5300 5750
-F 0 "#PWR107" H 5300 5500 50  0001 C CNN
+F 0 "#PWR0121" H 5300 5500 50  0001 C CNN
 F 1 "GND" H 5300 5600 50  0001 C CNN
 F 2 "" H 5300 5750 50  0001 C CNN
@@
 $EndComp
 $Comp
-L +12V #PWR104
+L +12V #PWR0122
 U 1 1 61244868
 P 4600 4850
-F 0 "#PWR104" H 4600 4700 50  0001 C CNN
+F 0 "#PWR0122" H 4600 4700 50  0001 C CNN
 F 1 "+12V" V 4600 5100 50  0000 C CNN
 F 2 "" H 4600 4850 50  0001 C CNN
@@
 Connection ~ 7200 5150
 $Comp
-L GND #PWR114
+L GND #PWR0123
 U 1 1 6124C7E1
 P 7200 5500
-F 0 "#PWR114" H 7200 5250 50  0001 C CNN
+F 0 "#PWR0123" H 7200 5250 50  0001 C CNN
 F 1 "GND" H 7200 5350 50  0001 C CNN
 F 2 "" H 7200 5500 50  0001 C CNN
@@
 	7200 5500 7200 5450
 $Comp
-L GND #PWR112
+L GND #PWR0124
 U 1 1 6124C940
 P 6650 5500
-F 0 "#PWR112" H 6650 5250 50  0001 C CNN
+F 0 "#PWR0124" H 6650 5250 50  0001 C CNN
 F 1 "GND" H 6650 5350 50  0001 C CNN
 F 2 "" H 6650 5500 50  0001 C CNN
@@
 $EndComp
 $Comp
-L +12V #PWR100
+L +12V #PWR0125
 U 1 1 6126FE6E
 P 2700 5250
-F 0 "#PWR100" H 2700 5100 50  0001 C CNN
+F 0 "#PWR0125" H 2700 5100 50  0001 C CNN
 F 1 "+12V" V 2700 5500 50  0000 C CNN
 F 2 "" H 2700 5250 50  0001 C CNN
@@
 $EndComp
 $Comp
-L GND #PWR99
+L GND #PWR0126
 U 1 1 612713A0
 P 2650 5850
-F 0 "#PWR99" H 2650 5600 50  0001 C CNN
+F 0 "#PWR0126" H 2650 5600 50  0001 C CNN
 F 1 "GND" H 2650 5700 50  0001 C CNN
 F 2 "" H 2650 5850 50  0001 C CNN
