File: PCB/KiCAD/RX_TX.sch (KiCad schematic (older format))
At the start: 13 parts, among them Q3 SI2301-TP, Q4 SI2301-TP

Commit message: PCB read works, layout BPF
Parts:
- C26, C27, C30: footprint Capacitors_SMD:C_0603_HandSoldering -> DragonFly:C_0603_HandSoldering
- D6, D7: footprint LEDs:LED_D3.0mm_Horizontal_O3.81mm_Z10.0mm -> DragonFly:LED_D3.0mm_Horizontal_O3.81mm_Z10.0mm
- Q3, Q4: footprint TO_SOT_Packages_SMD:SOT-23 -> DragonFly:SOT-23
- R13, R15, R32, R33: footprint Resistors_SMD:R_0603_HandSoldering -> DragonFly:R_0603_HandSoldering
Changed lines of the file:
@@
 F 0 "C26" H 4000 2300 50  0000 L CNN
 F 1 "100nF" H 4000 2400 50  0000 L CNN
-F 2 "Capacitors_SMD:C_0603_HandSoldering" H 4250 2300 50  0001 C CNN
+F 2 "DragonFly:C_0603_HandSoldering" H 4250 2300 50  0001 C CNN
 F 3 "" H 4250 2300 50  0000 C CNN
 	1    4250 2300
@@
 F 0 "R13" H 5050 3200 50  0000 L CNN
 F 1 "4.7K" H 5050 3300 50  0000 L CNN
-F 2 "Resistors_SMD:R_0603_HandSoldering" H 4950 3250 50  0001 C CNN
+F 2 "DragonFly:R_0603_HandSoldering" H 4950 3250 50  0001 C CNN
 F 3 "" H 4950 3250 50  0000 C CNN
 	1    4950 3250
@@
 F 0 "C27" H 5050 3200 50  0000 L CNN
 F 1 "100nF" H 4950 3300 50  0000 L CNN
-F 2 "Capacitors_SMD:C_0603_HandSoldering" H 5300 3250 50  0001 C CNN
+F 2 "DragonFly:C_0603_HandSoldering" H 5300 3250 50  0001 C CNN
 F 3 "" H 5300 3250 50  0000 C CNN
 	1    5300 3250
@@
 F 0 "C30" H 6500 2300 50  0000 L CNN
 F 1 "100nF" H 6400 2400 50  0000 L CNN
-F 2 "Capacitors_SMD:C_0603_HandSoldering" H 6750 2350 50  0001 C CNN
+F 2 "DragonFly:C_0603_HandSoldering" H 6750 2350 50  0001 C CNN
 F 3 "" H 6750 2350 50  0000 C CNN
 	1    6750 2350
@@
 $EndComp
 $Comp
-L GND #PWR72
+L GND #PWR071
 U 1 1 58DEEB52
 P 4950 3500
-F 0 "#PWR72" H 4950 3250 50  0001 C CNN
+F 0 "#PWR071" H 4950 3250 50  0001 C CNN
 F 1 "GND" H 4950 3350 50  0001 C CNN
 F 2 "" H 4950 3500 50  0000 C CNN
@@
 $EndComp
 $Comp
-L GND #PWR73
+L GND #PWR072
 U 1 1 58DEEB58
 P 5300 3500
-F 0 "#PWR73" H 5300 3250 50  0001 C CNN
+F 0 "#PWR072" H 5300 3250 50  0001 C CNN
 F 1 "GND" H 5300 3350 50  0001 C CNN
 F 2 "" H 5300 3500 50  0000 C CNN
@@
 F 0 "R15" H 6600 2350 50  0000 L CNN
 F 1 "4.7K" H 6600 2450 50  0000 L CNN
-F 2 "Resistors_SMD:R_0603_HandSoldering" H 6500 2350 50  0001 C CNN
+F 2 "DragonFly:R_0603_HandSoldering" H 6500 2350 50  0001 C CNN
 F 3 "" H 6500 2350 50  0000 C CNN
 	1    6500 2350
@@
 F 0 "Q3" H 5150 2400 50  0000 L CNN
 F 1 "SI2301-TP" H 5100 2500 50  0000 L CNN
-F 2 "TO_SOT_Packages_SMD:SOT-23" H 5050 2650 50  0001 C CNN
+F 2 "DragonFly:SOT-23" H 5050 2650 50  0001 C CNN
 F 3 "" H 4850 2550 50  0001 C CNN
 	1    4850 2550
@@
 $EndComp
 $Comp
-L +12V #PWR71
+L +12V #PWR073
 U 1 1 60FDEEDE
 P 3700 2100
-F 0 "#PWR71" H 3700 1950 50  0001 C CNN
+F 0 "#PWR073" H 3700 1950 50  0001 C CNN
 F 1 "+12V" V 3700 2350 50  0000 C CNN
 F 2 "" H 3700 2100 50  0001 C CNN
@@
 F 0 "Q4" V 6400 2100 50  0000 L CNN
 F 1 "SI2301-TP" V 6250 2050 50  0000 L CNN
-F 2 "TO_SOT_Packages_SMD:SOT-23" H 6200 2300 50  0001 C CNN
+F 2 "DragonFly:SOT-23" H 6200 2300 50  0001 C CNN
 F 3 "" H 6000 2200 50  0001 C CNN
 	1    6000 2200
@@
 Connection ~ 6500 2100
 $Comp
-L GND #PWR75
+L GND #PWR074
 U 1 1 60FDF676
 P 6500 2550
-F 0 "#PWR75" H 6500 2300 50  0001 C CNN
+F 0 "#PWR074" H 6500 2300 50  0001 C CNN
 F 1 "GND" H 6500 2400 50  0001 C CNN
 F 2 "" H 6500 2550 50  0000 C CNN
@@
 	6500 2550 6500 2450
 $Comp
-L GND #PWR76
+L GND #PWR075
 U 1 1 60FDF6C5
 P 6750 2550
-F 0 "#PWR76" H 6750 2300 50  0001 C CNN
+F 0 "#PWR075" H 6750 2300 50  0001 C CNN
 F 1 "GND" H 6750 2400 50  0001 C CNN
 F 2 "" H 6750 2550 50  0000 C CNN
@@
 F 0 "D6" V 6050 3300 50  0000 C CNN
 F 1 "RED" V 5950 3300 50  0000 C CNN
-F 2 "LEDs:LED_D3.0mm_Horizontal_O3.81mm_Z10.0mm" H 6000 3450 50  0001 C CNN
+F 2 "DragonFly:LED_D3.0mm_Horizontal_O3.81mm_Z10.0mm" H 6000 3450 50  0001 C CNN
 F 3 "" H 6000 3450 50  0001 C CNN
 	1    6000 3450
@@
 F 0 "R32" H 6100 3050 50  0000 L CNN
 F 1 "4.7K" H 6100 3150 50  0000 L CNN
-F 2 "Resistors_SMD:R_0603_HandSoldering" H 6000 3100 50  0001 C CNN
+F 2 "DragonFly:R_0603_HandSoldering" H 6000 3100 50  0001 C CNN
 F 3 "" H 6000 3100 50  0000 C CNN
 	1    6000 3100
@@
 $EndComp
 $Comp
-L GND #PWR74
+L GND #PWR076
 U 1 1 6106423B
 P 6000 3700
-F 0 "#PWR74" H 6000 3450 50  0001 C CNN
+F 0 "#PWR076" H 6000 3450 50  0001 C CNN
 F 1 "GND" H 6000 3550 50  0001 C CNN
 F 2 "" H 6000 3700 50  0000 C CNN
@@
 F 0 "R33" H 7750 2200 50  0000 L CNN
 F 1 "4.7K" H 7750 2300 50  0000 L CNN
-F 2 "Resistors_SMD:R_0603_HandSoldering" H 7650 2250 50  0001 C CNN
+F 2 "DragonFly:R_0603_HandSoldering" H 7650 2250 50  0001 C CNN
 F 3 "" H 7650 2250 50  0000 C CNN
 	1    7650 2250
@@
 F 0 "D7" V 7700 2400 50  0000 C CNN
 F 1 "GREEN" V 7600 2350 50  0000 C CNN
-F 2 "LEDs:LED_D3.0mm_Horizontal_O3.81mm_Z10.0mm" H 7650 2550 50  0001 C CNN
+F 2 "DragonFly:LED_D3.0mm_Horizontal_O3.81mm_Z10.0mm" H 7650 2550 50  0001 C CNN
 F 3 "" H 7650 2550 50  0001 C CNN
 	1    7650 2550
@@
 $EndComp
 $Comp
-L GND #PWR77
+L GND #PWR077
 U 1 1 61064CD8
 P 7650 2750
-F 0 "#PWR77" H 7650 2500 50  0001 C CNN
+F 0 "#PWR077" H 7650 2500 50  0001 C CNN
 F 1 "GND" H 7650 2600 50  0001 C CNN
 F 2 "" H 7650 2750 50  0000 C CNN
