File: PCB/KiCAD/RX_TX.sch (KiCad schematic (older format))
At the start: 13 parts, among them Q3 SI2301-TP, Q4 SI2301-TP

Commit message: PCB v1.0
Parts:
- C26, C27, C30: footprint DragonFly:C_0603_HandSoldering -> DragonFly:C_1206_0603
- R13, R15, R32, R33: footprint DragonFly:R_0603_HandSoldering -> DragonFly:R_1206_0603
Changed lines of the file:
@@
 F 0 "C26" H 4000 2300 50  0000 L CNN
 F 1 "100nF" H 4000 2400 50  0000 L CNN
-F 2 "DragonFly:C_0603_HandSoldering" H 4250 2300 50  0001 C CNN
+F 2 "DragonFly:C_1206_0603" H 4250 2300 50  0001 C CNN
 F 3 "" H 4250 2300 50  0000 C CNN
 	1    4250 2300
@@
 F 0 "R13" H 5050 3200 50  0000 L CNN
 F 1 "4.7K" H 5050 3300 50  0000 L CNN
-F 2 "DragonFly:R_0603_HandSoldering" H 4950 3250 50  0001 C CNN
+F 2 "DragonFly:R_1206_0603" H 4950 3250 50  0001 C CNN
 F 3 "" H 4950 3250 50  0000 C CNN
 	1    4950 3250
@@
 F 0 "C27" H 5050 3200 50  0000 L CNN
 F 1 "100nF" H 4950 3300 50  0000 L CNN
-F 2 "DragonFly:C_0603_HandSoldering" H 5300 3250 50  0001 C CNN
+F 2 "DragonFly:C_1206_0603" H 5300 3250 50  0001 C CNN
 F 3 "" H 5300 3250 50  0000 C CNN
 	1    5300 3250
@@
 F 0 "C30" H 6500 2300 50  0000 L CNN
 F 1 "100nF" H 6400 2400 50  0000 L CNN
-F 2 "DragonFly:C_0603_HandSoldering" H 6750 2350 50  0001 C CNN
+F 2 "DragonFly:C_1206_0603" H 6750 2350 50  0001 C CNN
 F 3 "" H 6750 2350 50  0000 C CNN
 	1    6750 2350
@@
 $EndComp
 $Comp
-L GND #PWR76
+L GND #PWR79
 U 1 1 58DEEB52
 P 4950 3500
-F 0 "#PWR76" H 4950 3250 50  0001 C CNN
+F 0 "#PWR79" H 4950 3250 50  0001 C CNN
 F 1 "GND" H 4950 3350 50  0001 C CNN
 F 2 "" H 4950 3500 50  0000 C CNN
@@
 $EndComp
 $Comp
-L GND #PWR77
+L GND #PWR80
 U 1 1 58DEEB58
 P 5300 3500
-F 0 "#PWR77" H 5300 3250 50  0001 C CNN
+F 0 "#PWR80" H 5300 3250 50  0001 C CNN
 F 1 "GND" H 5300 3350 50  0001 C CNN
 F 2 "" H 5300 3500 50  0000 C CNN
@@
 F 0 "R15" H 6600 2350 50  0000 L CNN
 F 1 "4.7K" H 6600 2450 50  0000 L CNN
-F 2 "DragonFly:R_0603_HandSoldering" H 6500 2350 50  0001 C CNN
+F 2 "DragonFly:R_1206_0603" H 6500 2350 50  0001 C CNN
 F 3 "" H 6500 2350 50  0000 C CNN
 	1    6500 2350
@@
 $EndComp
 $Comp
-L +12V #PWR75
+L +12V #PWR78
 U 1 1 60FDEEDE
 P 3700 2100
-F 0 "#PWR75" H 3700 1950 50  0001 C CNN
+F 0 "#PWR78" H 3700 1950 50  0001 C CNN
 F 1 "+12V" V 3700 2350 50  0000 C CNN
 F 2 "" H 3700 2100 50  0001 C CNN
@@
 Connection ~ 6500 2100
 $Comp
-L GND #PWR79
+L GND #PWR82
 U 1 1 60FDF676
 P 6500 2550
-F 0 "#PWR79" H 6500 2300 50  0001 C CNN
+F 0 "#PWR82" H 6500 2300 50  0001 C CNN
 F 1 "GND" H 6500 2400 50  0001 C CNN
 F 2 "" H 6500 2550 50  0000 C CNN
@@
 	6500 2550 6500 2450
 $Comp
-L GND #PWR80
+L GND #PWR83
 U 1 1 60FDF6C5
 P 6750 2550
-F 0 "#PWR80" H 6750 2300 50  0001 C CNN
+F 0 "#PWR83" H 6750 2300 50  0001 C CNN
 F 1 "GND" H 6750 2400 50  0001 C CNN
 F 2 "" H 6750 2550 50  0000 C CNN
@@
 F 0 "R32" H 6100 3050 50  0000 L CNN
 F 1 "4.7K" H 6100 3150 50  0000 L CNN
-F 2 "DragonFly:R_0603_HandSoldering" H 6000 3100 50  0001 C CNN
+F 2 "DragonFly:R_1206_0603" H 6000 3100 50  0001 C CNN
 F 3 "" H 6000 3100 50  0000 C CNN
 	1    6000 3100
@@
 $EndComp
 $Comp
-L GND #PWR78
+L GND #PWR81
 U 1 1 6106423B
 P 6000 3700
-F 0 "#PWR78" H 6000 3450 50  0001 C CNN
+F 0 "#PWR81" H 6000 3450 50  0001 C CNN
 F 1 "GND" H 6000 3550 50  0001 C CNN
 F 2 "" H 6000 3700 50  0000 C CNN
@@
 F 0 "R33" H 7750 2200 50  0000 L CNN
 F 1 "4.7K" H 7750 2300 50  0000 L CNN
-F 2 "DragonFly:R_0603_HandSoldering" H 7650 2250 50  0001 C CNN
+F 2 "DragonFly:R_1206_0603" H 7650 2250 50  0001 C CNN
 F 3 "" H 7650 2250 50  0000 C CNN
 	1    7650 2250
@@
 $EndComp
 $Comp
-L GND #PWR81
+L GND #PWR84
 U 1 1 61064CD8
 P 7650 2750
-F 0 "#PWR81" H 7650 2500 50  0001 C CNN
+F 0 "#PWR84" H 7650 2500 50  0001 C CNN
 F 1 "GND" H 7650 2600 50  0001 C CNN
 F 2 "" H 7650 2750 50  0000 C CNN
