File: PCB/KiCAD/DragonFly.kicad_pcb (KiCad board)
At the start: 2 copper layers, 120 x 93 mm, 136 parts, among them CON1 AVR-ISP-6, J1 USB_OTG, J2 JACK_TRS_3pins, J3 MIC, J7 Conn_Coaxial, K1 TQ2-12VDC, P4 CONN_01X01, P5 CONN_01X01, P6 CONN_01X01, P7 CONN_01X01, Q1 MMBFJ310LT1G, Q10 MMBT4401LT1G, Q11 BFG591, Q12 IRF610, Q2 MMBT2222A, Q3 SI2301-TP, Q4 SI2301-TP, Q5 MMBT2222A, Q6 MMBFJ310LT1G, T1 1_9, T2 1_4, T3 1_4, U1 ADE-1, U10 LD1117S33TR, U2 ATMEGA8-16AU, U3 ADuM1201CR, U4 LM78L06, U5 SA612, U6 FT232RL, U7 SI5351, U8 LM78L06, U9 SA612, Y1 8Mhz, Y2 8Mhz, Y3 8Mhz, Y4 8Mhz, Y5 8Mhz, Y6 8Mhz, Y7 8Mhz, Y8 27Mhz

Commit message: PCB home
Parts:
- added C54: 10...20pF, Capacitors_SMD:C_Trimmer_Voltronics_JZ, B.Cu at (148.8, 67.5)
- added C55: 10pF, DragonFly:C_1206_0603, F.Cu at (147.9, 47.0)
- added C56: 10pF, DragonFly:C_1206_0603, F.Cu at (148.8, 67.5)
- added C57: 100nF, Capacitors_SMD:C_0603_HandSoldering, F.Cu at (109.8, 102.2)
- added C58: 100nF, Capacitors_SMD:C_0603_HandSoldering, F.Cu at (130.8, 89.0)
- added C59: 62, Capacitors_SMD:C_0805, F.Cu at (116.8, 29.9)
- added C60: 10nF, Capacitors_SMD:C_0603_HandSoldering, F.Cu at (83.7, 27.8)
- added C61: 10µF, Capacitors_THT:CP_Radial_D5.0mm_P2.00mm, B.Cu at (74.0, 42.1)
- added C62: 47nF, DragonFly:C_1206_0603, F.Cu at (73.4, 24.6)
- added C63: 4.7nF, Capacitors_SMD:C_0603_HandSoldering, F.Cu at (61.7, 31.0)
- added C64: 100nF, Capacitors_SMD:C_0603_HandSoldering, F.Cu at (67.1, 24.2)
- added C65: 560pF, DragonFly:C_1206_0603, F.Cu at (151.3, 44.0)
- added C66: 560pF, DragonFly:C_1206_0603, F.Cu at (145.6, 67.5)
- added C67: 62, Capacitors_SMD:C_0805, F.Cu at (111.5, 29.8)
- added C68, C69: 470pF, Capacitors_THT:C_Disc_D6.0mm_W2.5mm_P5.00mm, F.Cu at (95.0, 123.1)
- added D10: BAT54S, TO_SOT_Packages_SMD:SOT-23, F.Cu at (132.2, 45.6)
- added D8: LL4148, Diodes_SMD:D_MiniMELF, F.Cu at (127.8, 96.2)
- added D9: BAT54S, TO_SOT_Packages_SMD:SOT-23, F.Cu at (135.2, 48.6)
- added J4: Conn_Coaxial, DragonFly:U.FL_Molex_MCRF_73412-0110_Vertical, B.Cu at (152.2, 42.2)
- added J5: Conn_Coaxial, DragonFly:U.FL_Molex_MCRF_73412-0110_Vertical, B.Cu at (151.7, 75.3)
- added L5: 1uH, Resistors_THT:R_Axial_DIN0411_L9.9mm_D3.6mm_P12.70mm_Horizontal, F.Cu at (95.0, 123.1)
- added L7: 31uH, Choke_Toroid_ThroughHole:Choke_Toroid_5x10mm_Vertical, B.Cu at (143.8, 58.0)
- added R29, R30: 10K, DragonFly:R_1206_0603, F.Cu at (95.0, 123.1)
- added R34: 3.3k, DragonFly:R_1206_0603, F.Cu at (113.6, 105.3)
- added R36: 3.3k, DragonFly:R_1206_0603, F.Cu at (67.3, 38.2)
- added R37: 1k, Resistors_SMD:R_0603_HandSoldering, F.Cu at (75.0, 31.8)
- added R38: 15k, Resistors_SMD:R_0603_HandSoldering, F.Cu at (75.0, 29.6)
- added R39: 100R, DragonFly:R_1206_0603, F.Cu at (59.6, 26.1)
- added R40: 560, DragonFly:R_1206_0603, F.Cu at (56.1, 26.2)
- added RV2: 1k, Potentiometers:Potentiometer_Trimmer_Piher_PT-6v_Horizontal, B.Cu at (74.0, 47.5)
- added T4: Transformer_1P_2S, DragonFly:HF12, B.Cu at (128.3, 52.6)
- added T5: Transformer_1P_2S, DragonFly:HF12, B.Cu at (139.4, 47.5)
- added Y10: 8Mhz, DragonFly:Crystal_HC49-U_Vertical, B.Cu at (114.1, 27.4)
- added Y9: 8Mhz, DragonFly:Crystal_HC49-U_Vertical, B.Cu at (119.3, 32.3)
- C43: value 10pF -> 100nF; footprint DragonFly:C_1206_0603 -> Capacitors_SMD:C_0603_HandSoldering
- C44: value 390pF -> 1nF
- C45: value 10pF -> 10...20pF; footprint DragonFly:C_1206_0603 -> Capacitors_SMD:C_Trimmer_Voltronics_JZ; moved to B.Cu
- L6: value 52uH -> 31uH; footprint LCSDR:Resistor_Horizontal_RM10mm -> Choke_Toroid_ThroughHole:Choke_Toroid_5x10mm_Vertical
- U1: value ADE-1 -> NE5532; footprint DragonFly:ADE-1H -> Housings_SOIC:SOIC-8_3.9x4.9mm_Pitch1.27mm
- moved C44 128.5 mm to (145.3, 56.7)
- moved C45 108.0 mm to (147.9, 47.0), turned to 0 degrees
- moved L6 106.1 mm to (143.8, 50.2), turned to 0 degrees
- moved C43 61.5 mm to (61.5, 98.2), turned to 270 degrees
- moved U1 53.7 mm to (69.0, 31.4), turned to 90 degrees
- moved C9 42.7 mm to (143.2, 27.4)
- moved D2 40.7 mm to (152.2, 25.1)
- moved R12 40.5 mm to (143.2, 24.9)
- moved C6 39.2 mm to (152.2, 29.3)
- moved T2 38.5 mm to (146.6, 29.9)
- moved R5 38.2 mm to (83.5, 42.1), turned to 0 degrees
- moved R10 37.4 mm to (152.2, 34.1), turned to 270 degrees
- moved Q1 37.3 mm to (147.8, 33.0)
- moved C8 35.8 mm to (121.9, 29.9)
- moved C4 35.8 mm to (132.2, 29.9)
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Connections:
- C43 pad 1: Net-(C43-Pad1) -> +3V3
- C43 pad 2: Net-(C43-Pad2) -> GND
- C44 pad 1: Net-(C43-Pad2) -> Net-(C44-Pad1)
- C45 pad 1: Net-(C43-Pad2) -> BPF
- C45 pad 2: (no net) -> Net-(C45-Pad2)
- J7 pad 1: Net-(E1-Pad1) -> Net-(C69-Pad1)
- K1 pad 1: (no net) -> +12V
- K1 pad 10: (no net) -> Net-(D8-Pad2)
- K1 pad 3: Net-(E1-Pad1) -> Net-(C68-Pad1)
- K1 pad 8: (no net) -> Net-(C54-Pad2)
- L6 pad 1: BPF -> Net-(C45-Pad2)
- L6 pad 2: Net-(C43-Pad1) -> Net-(C44-Pad1)
- Q5 pad 1: (no net) -> Net-(Q5-Pad1)
- Q5 pad 3: (no net) -> Net-(D8-Pad2)
- U1 pad 1: Net-(Q2-Pad3) -> Net-(R36-Pad1)
- U1 pad 2: Net-(C1-Pad2) -> Net-(C61-Pad1)
- U1 pad 3: Net-(C2-Pad2) -> Net-(C60-Pad2)
- U1 pad 5: GND -> Net-(C63-Pad2)
- U1 pad 6: +12V -> Net-(C62-Pad1)
- U5 pad 5: Net-(C23-Pad1) -> Net-(C60-Pad2)
- Y5 pad 1: Net-(C8-Pad2) -> Net-(C67-Pad2)
- Y6 pad 1: Net-(C8-Pad2) -> Net-(C67-Pad2)
Routing:
- removed copper zone on B.Cu, net GND
