File: PCB/KiCAD/DragonFly.sch (KiCad schematic (older format))
At the start: 33 parts, among them Q1 MMBFJ310LT1G, T2 1_4, Y1 8Mhz, Y10 8Mhz, Y11 8Mhz, Y12 8Mhz, Y2 8Mhz, Y3 8Mhz, Y4 8Mhz, Y5 8Mhz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

Commit message: PCB v1.0
Parts:
- C10: footprint Capacitors_SMD:C_0603_HandSoldering -> DragonFly:C_1206_0603
- C6, C9: value 100nF -> 10nF
- R2: footprint DragonFly:R_0603_HandSoldering -> DragonFly:R_1206_0603
Changed lines of the file:
@@
 P 3050 3150
 F 0 "C6" H 3150 3100 50  0000 L CNN
-F 1 "100nF" H 3150 3200 50  0000 L CNN
+F 1 "10nF" H 3150 3200 50  0000 L CNN
 F 2 "DragonFly:C_0603_HandSoldering" H 3050 3150 50  0001 C CNN
 F 3 "" H 3050 3150 50  0000 C CNN
@@
 P 3250 2400
 F 0 "C9" V 3050 2350 50  0000 L CNN
-F 1 "100nF" V 3150 2350 50  0000 L CNN
+F 1 "10nF" V 3150 2350 50  0000 L CNN
 F 2 "Capacitors_SMD:C_0603_HandSoldering" H 3250 2400 50  0001 C CNN
 F 3 "" H 3250 2400 50  0000 C CNN
@@
 F 0 "R2" H 6650 3800 50  0000 L CNN
 F 1 "1k" H 6650 3700 50  0000 L CNN
-F 2 "DragonFly:R_0603_HandSoldering" H 6550 3750 50  0001 C CNN
+F 2 "DragonFly:R_1206_0603" H 6550 3750 50  0001 C CNN
 F 3 "" H 6550 3750 50  0000 C CNN
 	1    6550 3750
@@
 F 0 "C10" H 6500 3700 50  0000 L CNN
 F 1 "100nF" H 6400 3800 50  0000 L CNN
-F 2 "Capacitors_SMD:C_0603_HandSoldering" H 6300 3750 50  0001 C CNN
+F 2 "DragonFly:C_1206_0603" H 6300 3750 50  0001 C CNN
 F 3 "" H 6300 3750 50  0000 C CNN
 	1    6300 3750
