File: PCB/KiCAD/IF.sch (KiCad schematic (older format))
At the start: 23 parts, among them J2 JACK_TRS_3pins, P4 CONN_01X01, P5 CONN_01X01, P6 CONN_01X01, P7 CONN_01X01, Q6 MMBFJ310LT1G, U4 LM78L06, U5 SA612

Commit message: PCB home
Parts:
- added C60: 10nF, Capacitors_SMD:C_0603_HandSoldering, symbol C_Small
- added C61: 10µF, Capacitors_THT:CP_Radial_D5.0mm_P2.00mm, symbol CP_Small
- added C62: 47nF, DragonFly:C_1206_0603, symbol C_Small
- added C63: 4.7nF, Capacitors_SMD:C_0603_HandSoldering, symbol C_Small
- added C64: 100nF, Capacitors_SMD:C_0603_HandSoldering, symbol C_Small
- added R36: 3.3k, DragonFly:R_1206_0603, symbol R_Small
- added R37: 1k, Resistors_SMD:R_0603_HandSoldering, symbol R_Small
- added R38: 15k, Resistors_SMD:R_0603_HandSoldering, symbol R_Small
- added R39: 100R, DragonFly:R_1206_0603, symbol R_Small
- added R40: 560, DragonFly:R_1206_0603, symbol R_Small
- added RV2: 1k, Potentiometers:Potentiometer_Trimmer_Piher_PT-6v_Horizontal, symbol POT
- added U1: NE5532, Housings_SOIC:SOIC-8_3.9x4.9mm_Pitch1.27mm, symbol NE5532
Connections:
- net GND: now also C60.1, C63.1, C64.1, RV2.2, RV2.3, U1.4 (V-), U1.4 (V-)
- net RX_12V: now also R39.1
- net at U5.5 (OUT_B): now also C60.2, U1.3 (+); no longer C23.1
- new net: C23.1, R40.1
- new net: R36.1, R37.2, U1.1
- new net: C61.1, R36.2, U1.2 (-)
- new net: C64.2, R39.2, U1.8 (V+), U1.8 (V+)
- new net: C63.2, R38.1, U1.5 (+)
- new net: C62.1, R40.2, U1.6 (-), U1.7
- new net: C62.2, R37.1, R38.2
- new net: C61.2, RV2.1
Other:
- moved on the sheet: C23, J2
