File: PCB/KiCAD/IF.sch (KiCad schematic (older format))
At the start: 42 parts, among them J2 JACK_TRS_3pins, P4 CONN_01X01, P5 CONN_01X01, P6 CONN_01X01, P7 CONN_01X01, Q2 2N7002, Q6 MMBFJ310L, U1 NE5532, U4 L78L06_TO92, U5 SA612

Commit message: PCB v1.0
Parts:
- added Q8: 2N7002, DragonFly:SOT-23, symbol 2N7002
- added R43: 3.3K, DragonFly:R_1206_0603, symbol R_Small
- C20, C24, C25, C28, C31, C76: footprint DragonFly:C_0603_HandSoldering -> DragonFly:C_1206_0603
- C29: value 100nF -> 10nF
- C58, C78: footprint Capacitors_SMD:C_0603_HandSoldering -> DragonFly:C_1206_0603
- R17: footprint DragonFly:R_0603_HandSoldering -> DragonFly:R_1206_0603
Connections:
- net GND: now also Q8.2 (S)
- net at C77.1, D9.2 (K), Q2.1 (G)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: now also Q8.3 (D)
- new net: Q8.1 (G), R43.2
- new net AGC_OFF: R43.1
Changed lines of the file:
@@
 $EndComp
 $Comp
-L GND #PWR71
+L GND #PWR74
 U 1 1 58912103
 P 10550 700
-F 0 "#PWR71" H 10550 450 50  0001 C CNN
+F 0 "#PWR74" H 10550 450 50  0001 C CNN
 F 1 "GND" H 10550 550 50  0001 C CNN
 F 2 "" H 10550 700 50  0000 C CNN
@@
 $EndComp
 $Comp
-L GND #PWR72
+L GND #PWR75
 U 1 1 58912546
 P 10550 900
-F 0 "#PWR72" H 10550 650 50  0001 C CNN
+F 0 "#PWR75" H 10550 650 50  0001 C CNN
 F 1 "GND" H 10550 750 50  0001 C CNN
 F 2 "" H 10550 900 50  0000 C CNN
@@
 $EndComp
 $Comp
-L GND #PWR73
+L GND #PWR76
 U 1 1 58912989
 P 10550 1100
-F 0 "#PWR73" H 10550 850 50  0001 C CNN
+F 0 "#PWR76" H 10550 850 50  0001 C CNN
 F 1 "GND" H 10550 950 50  0001 C CNN
 F 2 "" H 10550 1100 50  0000 C CNN
@@
 $EndComp
 $Comp
-L GND #PWR74
+L GND #PWR77
 U 1 1 589132CC
 P 10550 1300
-F 0 "#PWR74" H 10550 1050 50  0001 C CNN
+F 0 "#PWR77" H 10550 1050 50  0001 C CNN
 F 1 "GND" H 10550 1150 50  0001 C CNN
 F 2 "" H 10550 1300 50  0000 C CNN
@@
 $EndComp
 $Comp
-L GND #PWR55
+L GND #PWR57
 U 1 1 58AF70A6
 P 3000 1600
-F 0 "#PWR55" H 3000 1350 50  0001 C CNN
+F 0 "#PWR57" H 3000 1350 50  0001 C CNN
 F 1 "GND" H 3000 1450 50  0001 C CNN
 F 2 "" H 3000 1600 50  0000 C CNN
@@
 F 0 "C28" V 2700 2350 50  0000 L CNN
 F 1 "100nF" V 2800 2350 50  0000 L CNN
-F 2 "DragonFly:C_0603_HandSoldering" H 2950 2500 50  0001 C CNN
+F 2 "DragonFly:C_1206_0603" H 2950 2500 50  0001 C CNN
 F 3 "" H 2950 2500 50  0000 C CNN
 	1    2950 2500
@@
 $EndComp
 $Comp
-L GND #PWR51
+L GND #PWR53
 U 1 1 58B15E5F
 P 2250 3300
-F 0 "#PWR51" H 2250 3050 50  0001 C CNN
+F 0 "#PWR53" H 2250 3050 50  0001 C CNN
 F 1 "GND" H 2250 3150 50  0001 C CNN
 F 2 "" H 2250 3300 50  0000 C CNN
@@
 $EndComp
 $Comp
-L GND #PWR48
+L GND #PWR50
 U 1 1 58B0B2EB
 P 1400 3300
-F 0 "#PWR48" H 1400 3050 50  0001 C CNN
+F 0 "#PWR50" H 1400 3050 50  0001 C CNN
 F 1 "GND" H 1400 3150 50  0001 C CNN
 F 2 "" H 1400 3300 50  0000 C CNN
@@
 F 0 "C24" H 2050 1400 50  0000 L CNN
 F 1 "100nF" H 2050 1500 50  0000 L CNN
-F 2 "DragonFly:C_0603_HandSoldering" H 1950 1450 50  0001 C CNN
+F 2 "DragonFly:C_1206_0603" H 1950 1450 50  0001 C CNN
 F 3 "" H 1950 1450 50  0000 C CNN
 	1    1950 1450
@@
 $EndComp
 $Comp
-L GND #PWR49
+L GND #PWR51
 U 1 1 58B0BE25
 P 1950 1550
-F 0 "#PWR49" H 1950 1300 50  0001 C CNN
+F 0 "#PWR51" H 1950 1300 50  0001 C CNN
 F 1 "GND" H 1950 1400 50  0001 C CNN
 F 2 "" H 1950 1550 50  0000 C CNN
@@
 F 0 "R17" H 1200 3250 50  0000 L CNN
 F 1 "10k" H 1200 3150 50  0000 L CNN
-F 2 "DragonFly:R_0603_HandSoldering" H 1400 3200 50  0001 C CNN
+F 2 "DragonFly:R_1206_0603" H 1400 3200 50  0001 C CNN
 F 3 "" H 1400 3200 50  0000 C CNN
 	1    1400 3200
@@
 $EndComp
 $Comp
-L GND #PWR50
+L GND #PWR52
 U 1 1 58B02D08
 P 2100 3300
-F 0 "#PWR50" H 2100 3050 50  0001 C CNN
+F 0 "#PWR52" H 2100 3050 50  0001 C CNN
 F 1 "GND" H 2100 3150 50  0001 C CNN
 F 2 "" H 2100 3300 50  0000 C CNN
@@
 $EndComp
 $Comp
-L GND #PWR53
+L GND #PWR55
 U 1 1 58B09A3F
 P 2700 2750
-F 0 "#PWR53" H 2700 2500 50  0001 C CNN
+F 0 "#PWR55" H 2700 2500 50  0001 C CNN
 F 1 "GND" H 2700 2600 50  0001 C CNN
 F 2 "" H 2700 2750 50  0000 C CNN
@@
 P 3100 2100
 F 0 "C29" H 2850 2050 50  0000 L CNN
-F 1 "100nF" H 2750 2150 50  0000 L CNN
+F 1 "10nF" H 2750 2150 50  0000 L CNN
 F 2 "Capacitors_SMD:C_0603_HandSoldering" H 3100 2100 50  0001 C CNN
 F 3 "" H 3100 2100 50  0000 C CNN
@@
 	4300 2400 4150 2400
 $Comp
-L GND #PWR56
+L GND #PWR58
 U 1 1 58B399E4
 P 3650 1600
-F 0 "#PWR56" H 3650 1350 50  0001 C CNN
+F 0 "#PWR58" H 3650 1350 50  0001 C CNN
 F 1 "GND" H 3650 1450 50  0001 C CNN
 F 2 "" H 3650 1600 50  0000 C CNN
@@
 $EndComp
 $Comp
-L GND #PWR58
+L GND #PWR60
 U 1 1 58B39C92
 P 3850 1600
-F 0 "#PWR58" H 3850 1350 50  0001 C CNN
+F 0 "#PWR60" H 3850 1350 50  0001 C CNN
 F 1 "GND" H 3850 1450 50  0001 C CNN
 F 2 "" H 3850 1600 50  0000 C CNN
@@
 $EndComp
 $Comp
-L GND #PWR54
+L GND #PWR56
 U 1 1 58B3CA01
 P 2850 2500
-F 0 "#PWR54" H 2850 2250 50  0001 C CNN
+F 0 "#PWR56" H 2850 2250 50  0001 C CNN
 F 1 "GND" H 2850 2350 50  0001 C CNN
 F 2 "" H 2850 2500 50  0000 C CNN
@@
 F 0 "C25" H 2200 3150 50  0000 L CNN
 F 1 "100nF" H 2200 3250 50  0000 L CNN
-F 2 "DragonFly:C_0603_HandSoldering" H 2100 3200 50  0001 C CNN
+F 2 "DragonFly:C_1206_0603" H 2100 3200 50  0001 C CNN
 F 3 "" H 2100 3200 50  0000 C CNN
 	1    2100 3200
@@
 $EndComp
 $Comp
-L GND #PWR62
+L GND #PWR65
 U 1 1 60FB6B9C
 P 4900 1800
-F 0 "#PWR62" H 4900 1550 50  0001 C CNN
+F 0 "#PWR65" H 4900 1550 50  0001 C CNN
 F 1 "GND" H 4900 1650 50  0001 C CNN
 F 2 "" H 4900 1800 50  0000 C CNN
@@
 F 0 "C20" V 4250 2400 50  0000 L CNN
 F 1 "100nF" V 4350 2400 50  0000 L CNN
-F 2 "DragonFly:C_0603_HandSoldering" H 4450 2500 50  0001 C CNN
+F 2 "DragonFly:C_1206_0603" H 4450 2500 50  0001 C CNN
 F 3 "" H 4450 2500 50  0000 C CNN
 	1    4450 2500
@@
 $EndComp
 $Comp
-L GND #PWR60
+L GND #PWR63
 U 1 1 60FB7F45
 P 4550 2500
-F 0 "#PWR60" H 4550 2250 50  0001 C CNN
+F 0 "#PWR63" H 4550 2250 50  0001 C CNN
 F 1 "GND" H 4550 2350 50  0001 C CNN
 F 2 "" H 4550 2500 50  0000 C CNN
@@
 $EndComp
 $Comp
-L GND #PWR70
+L GND #PWR73
 U 1 1 60FB9C6F
 P 9550 3900
-F 0 "#PWR70" H 9550 3650 50  0001 C CNN
+F 0 "#PWR73" H 9550 3650 50  0001 C CNN
 F 1 "GND" H 9550 3750 50  0001 C CNN
 F 2 "" H 9550 3900 50  0000 C CNN
@@
 F 0 "C31" H 3750 1450 50  0000 L CNN
 F 1 "100nF" H 3750 1550 50  0000 L CNN
-F 2 "DragonFly:C_0603_HandSoldering" H 3650 1500 50  0001 C CNN
+F 2 "DragonFly:C_1206_0603" H 3650 1500 50  0001 C CNN
 F 3 "" H 3650 1500 50  0000 C CNN
 	1    3650 1500
@@
 Connection ~ 6700 3300
 $Comp
-L GND #PWR69
+L GND #PWR72
 U 1 1 6123D132
 P 7850 3700
-F 0 "#PWR69" H 7850 3450 50  0001 C CNN
+F 0 "#PWR72" H 7850 3450 50  0001 C CNN
 F 1 "GND" H 7850 3550 50  0001 C CNN
 F 2 "" H 7850 3700 50  0000 C CNN
@@
 $EndComp
 $Comp
-L GND #PWR63
+L GND #PWR66
 U 1 1 61240985
 P 4950 3550
-F 0 "#PWR63" H 4950 3300 50  0001 C CNN
+F 0 "#PWR66" H 4950 3300 50  0001 C CNN
 F 1 "GND" H 4950 3400 50  0001 C CNN
 F 2 "" H 4950 3550 50  0000 C CNN
@@
 $EndComp
 $Comp
-L GND #PWR66
+L GND #PWR69
 U 1 1 61240A0C
 P 5600 3600
-F 0 "#PWR66" H 5600 3350 50  0001 C CNN
+F 0 "#PWR69" H 5600 3350 50  0001 C CNN
 F 1 "GND" H 5600 3450 50  0001 C CNN
 F 2 "" H 5600 3600 50  0000 C CNN
@@
 Connection ~ 7200 3200
 $Comp
-L GND #PWR68
+L GND #PWR71
 U 1 1 61241D9A
 P 7200 3500
-F 0 "#PWR68" H 7200 3250 50  0001 C CNN
+F 0 "#PWR71" H 7200 3250 50  0001 C CNN
 F 1 "GND" H 7200 3350 50  0001 C CNN
 F 2 "" H 7200 3500 50  0000 C CNN
@@
 	5250 4150 5250 4250
 $Comp
-L GND #PWR65
+L GND #PWR68
 U 1 1 61243457
 P 5250 4650
-F 0 "#PWR65" H 5250 4400 50  0001 C CNN
+F 0 "#PWR68" H 5250 4400 50  0001 C CNN
 F 1 "GND" H 5250 4500 50  0001 C CNN
 F 2 "" H 5250 4650 50  0000 C CNN
@@
 F 0 "C58" V 5100 2750 50  0000 L CNN
 F 1 "100nF" V 5200 2750 50  0000 L CNN
-F 2 "Capacitors_SMD:C_0603_HandSoldering" H 5300 2850 50  0001 C CNN
+F 2 "DragonFly:C_1206_0603" H 5300 2850 50  0001 C CNN
 F 3 "" H 5300 2850 50  0000 C CNN
 	1    5300 2850
@@
 	7850 2850 7850 3000
 $Comp
-L GND #PWR64
+L GND #PWR67
 U 1 1 61244C87
 P 5100 2850
-F 0 "#PWR64" H 5100 2600 50  0001 C CNN
+F 0 "#PWR67" H 5100 2600 50  0001 C CNN
 F 1 "GND" H 5100 2700 50  0001 C CNN
 F 2 "" H 5100 2850 50  0000 C CNN
@@
 	8550 5550 6150 5550
 $Comp
-L GND #PWR67
+L GND #PWR70
 U 1 1 612EB84D
 P 5600 5850
-F 0 "#PWR67" H 5600 5600 50  0001 C CNN
+F 0 "#PWR70" H 5600 5600 50  0001 C CNN
 F 1 "GND" H 5600 5700 50  0001 C CNN
 F 2 "" H 5600 5850 50  0000 C CNN
@@
 F 0 "C78" V 6250 5500 50  0000 L CNN
 F 1 "100nF" V 6150 5400 50  0000 L CNN
-F 2 "Capacitors_SMD:C_0603_HandSoldering" H 6050 5550 50  0001 C CNN
+F 2 "DragonFly:C_1206_0603" H 6050 5550 50  0001 C CNN
 F 3 "" H 6050 5550 50  0001 C CNN
 	1    6050 5550
@@
 $EndComp
 $Comp
-L GND #PWR61
+L GND #PWR64
 U 1 1 612EC5A9
 P 4850 5500
-F 0 "#PWR61" H 4850 5250 50  0001 C CNN
+F 0 "#PWR64" H 4850 5250 50  0001 C CNN
 F 1 "GND" H 4850 5350 50  0001 C CNN
 F 2 "" H 4850 5500 50  0000 C CNN
@@
 $EndComp
 $Comp
-L GND #PWR59
+L GND #PWR62
 U 1 1 612ED251
 P 4400 5500
-F 0 "#PWR59" H 4400 5250 50  0001 C CNN
+F 0 "#PWR62" H 4400 5250 50  0001 C CNN
 F 1 "GND" H 4400 5350 50  0001 C CNN
 F 2 "" H 4400 5500 50  0000 C CNN
@@
 $EndComp
 $Comp
-L GND #PWR57
+L GND #PWR59
 U 1 1 612ED845
 P 3750 5350
-F 0 "#PWR57" H 3750 5100 50  0001 C CNN
+F 0 "#PWR59" H 3750 5100 50  0001 C CNN
 F 1 "GND" H 3750 5200 50  0001 C CNN
 F 2 "" H 3750 5350 50  0000 C CNN
@@
 F 0 "C76" H 2600 4250 50  0000 L CNN
 F 1 "100nF" H 2600 4350 50  0000 L CNN
-F 2 "DragonFly:C_0603_HandSoldering" H 2500 4300 50  0001 C CNN
+F 2 "DragonFly:C_1206_0603" H 2500 4300 50  0001 C CNN
 F 3 "" H 2500 4300 50  0000 C CNN
 	1    2500 4300
@@
 $EndComp
 $Comp
-L GND #PWR52
+L GND #PWR54
 U 1 1 612EFA19
 P 2500 4400
-F 0 "#PWR52" H 2500 4150 50  0001 C CNN
+F 0 "#PWR54" H 2500 4150 50  0001 C CNN
 F 1 "GND" H 2500 4250 50  0001 C CNN
 F 2 "" H 2500 4400 50  0000 C CNN
@@
 	1    0    0    -1
 $EndComp
+$Comp
+L 2N7002 Q8
+U 1 1 612FE383
+P 4100 5850
+F 0 "Q8" H 4300 5925 50  0000 L CNN
+F 1 "2N7002" H 4300 5850 50  0000 L CNN
+F 2 "DragonFly:SOT-23" H 4300 5775 50  0001 L CIN
+F 3 "" H 4100 5850 50  0001 L CNN
+	1    4100 5850
+	1    0    0    -1
+$EndComp
+$Comp
+L GND #PWR61
+U 1 1 612FE450
+P 4200 6050
+F 0 "#PWR61" H 4200 5800 50  0001 C CNN
+F 1 "GND" H 4200 5900 50  0001 C CNN
+F 2 "" H 4200 6050 50  0000 C CNN
+F 3 "" H 4200 6050 50  0000 C CNN
+	1    4200 6050
+	1    0    0    -1
+$EndComp
+Wire Wire Line
+	4200 5650 4200 5150
+Connection ~ 4200 5150
+$Comp
+L R_Small R43
+U 1 1 612FE5CF
+P 3600 5850
+F 0 "R43" V 3800 5900 50  0000 L CNN
+F 1 "3.3K" V 3700 5800 50  0000 L CNN
+F 2 "DragonFly:R_1206_0603" H 3600 5850 50  0001 C CNN
+F 3 "" H 3600 5850 50  0001 C CNN
+	1    3600 5850
+	0    -1   -1   0
+$EndComp
+Wire Wire Line
+	3700 5850 3900 5850
+Wire Wire Line
+	3500 5850 3050 5850
+Text GLabel 3050 5850 0    60   Input ~ 0
+AGC_OFF
 $EndSCHEMATC
