File: PCB/KiCAD/IF_SA612_TX.sch (KiCad schematic (older format))
At the start: 19 parts, among them J3 MIC, Q10 MMBT4401LT1G, U8 LM78L06, U9 SA612

Commit message: PCB progress, IF TX, IF RX, PowerSupply Jack
Parts:
- C40: value 100µF -> 1µF; footprint DragonFly:CP_Radial_D6.3mm_P2.50mm -> DragonFly:CP_Radial_D4.0mm_P2.00mm
Changed lines of the file:
@@
 P 5300 1400
 F 0 "C40" H 5400 1400 50  0000 L CNN
-F 1 "100µF" H 5400 1300 50  0000 L CNN
-F 2 "DragonFly:CP_Radial_D6.3mm_P2.50mm" H 5300 1400 50  0001 C CNN
+F 1 "1µF" H 5400 1300 50  0000 L CNN
+F 2 "DragonFly:CP_Radial_D4.0mm_P2.00mm" H 5300 1400 50  0001 C CNN
 F 3 "" H 5300 1400 50  0000 C CNN
 	1    5300 1400

Commit message: mixer schema is done, pcb progress, fix 78l06 issue
Parts:
- removed U8: LM78L06, DragonFly:TO-92_Molded_Wide_Oval, symbol LM78L05
- added U8: L78L06_TO92, DragonFly:TO-92_Molded_Wide_Oval, symbol L78L06_TO92
Connections:
- net GND: now also U8.2 (GND)
- net TX_12V: now also U8.3 (VI)
- net TX_6V: now also U8.1 (VO)
Changed lines of the file:
@@
 $EndDescr
 $Comp
-L GND #PWR82
+L GND #PWR77
 U 1 1 58E1AB18
 P 1750 2050
-F 0 "#PWR82" H 1750 1800 50  0001 C CNN
+F 0 "#PWR77" H 1750 1800 50  0001 C CNN
 F 1 "GND" H 1750 1900 50  0001 C CNN
 F 2 "" H 1750 2050 50  0000 C CNN
@@
 $EndComp
 $Comp
-L GND #PWR84
+L GND #PWR79
 U 1 1 58E1AB3A
 P 2950 4000
-F 0 "#PWR84" H 2950 3750 50  0001 C CNN
+F 0 "#PWR79" H 2950 3750 50  0001 C CNN
 F 1 "GND" H 2950 3850 50  0001 C CNN
 F 2 "" H 2950 4000 50  0000 C CNN
@@
 $EndComp
 $Comp
-L GND #PWR83
+L GND #PWR78
 U 1 1 58E1AB40
 P 2200 4000
-F 0 "#PWR83" H 2200 3750 50  0001 C CNN
+F 0 "#PWR78" H 2200 3750 50  0001 C CNN
 F 1 "GND" H 2200 3850 50  0001 C CNN
 F 2 "" H 2200 4000 50  0000 C CNN
@@
 $EndComp
 $Comp
-L LM78L05 U8
-U 1 1 58E1AB63
-P 3250 1200
-F 0 "U8" H 3250 1500 50  0000 C CNN
-F 1 "LM78L06" H 3250 1400 50  0000 C CNN
-F 2 "DragonFly:TO-92_Molded_Wide_Oval" H 3250 1200 50  0001 C CNN
-F 3 "" H 3250 1200 50  0000 C CNN
-	1    3250 1200
-	1    0    0    -1
-$EndComp
-$Comp
-L GND #PWR86
+L GND #PWR81
 U 1 1 58E1AB6A
 P 3250 1450
-F 0 "#PWR86" H 3250 1200 50  0001 C CNN
+F 0 "#PWR81" H 3250 1200 50  0001 C CNN
 F 1 "GND" H 3250 1300 50  0001 C CNN
 F 2 "" H 3250 1450 50  0000 C CNN
@@
 $EndComp
 $Comp
-L GND #PWR90
+L GND #PWR85
 U 1 1 58E1AB77
 P 5100 2050
-F 0 "#PWR90" H 5100 1800 50  0001 C CNN
+F 0 "#PWR85" H 5100 1800 50  0001 C CNN
 F 1 "GND" H 5100 1900 50  0001 C CNN
 F 2 "" H 5100 2050 50  0000 C CNN
@@
 $EndComp
 $Comp
-L GND #PWR89
+L GND #PWR84
 U 1 1 58E1AB7D
 P 4950 2850
-F 0 "#PWR89" H 4950 2600 50  0001 C CNN
+F 0 "#PWR84" H 4950 2600 50  0001 C CNN
 F 1 "GND" H 4950 2700 50  0001 C CNN
 F 2 "" H 4950 2850 50  0000 C CNN
@@
 $EndComp
 $Comp
-L GND #PWR88
+L GND #PWR83
 U 1 1 58E1ABAE
 P 4800 1500
-F 0 "#PWR88" H 4800 1250 50  0001 C CNN
+F 0 "#PWR83" H 4800 1250 50  0001 C CNN
 F 1 "GND" H 4800 1350 50  0001 C CNN
 F 2 "" H 4800 1500 50  0000 C CNN
@@
 $EndComp
 $Comp
-L GND #PWR91
+L GND #PWR86
 U 1 1 58E1ABB4
 P 5300 1500
-F 0 "#PWR91" H 5300 1250 50  0001 C CNN
+F 0 "#PWR86" H 5300 1250 50  0001 C CNN
 F 1 "GND" H 5300 1350 50  0001 C CNN
 F 2 "" H 5300 1500 50  0000 C CNN
@@
 Connection ~ 5950 2250
 $Comp
-L GND #PWR92
+L GND #PWR87
 U 1 1 58E1ABEC
 P 5850 2400
-F 0 "#PWR92" H 5850 2150 50  0001 C CNN
+F 0 "#PWR87" H 5850 2150 50  0001 C CNN
 F 1 "GND" H 5850 2250 50  0001 C CNN
 F 2 "" H 5850 2400 50  0000 C CNN
@@
 	5850 2350 6050 2350
 $Comp
-L GND #PWR93
+L GND #PWR88
 U 1 1 58E1ABF4
 P 5850 2950
-F 0 "#PWR93" H 5850 2700 50  0001 C CNN
+F 0 "#PWR88" H 5850 2700 50  0001 C CNN
 F 1 "GND" H 5850 2800 50  0001 C CNN
 F 2 "" H 5850 2950 50  0000 C CNN
@@
 TX_6V
 Wire Wire Line
-	1600 1150 2850 1150
+	1600 1150 2950 1150
 Connection ~ 2650 1150
 Wire Wire Line
@@
 	2950 3800 2950 4000
 $Comp
-L GND #PWR87
+L GND #PWR82
 U 1 1 60FE7FDF
 P 3500 4250
-F 0 "#PWR87" H 3500 4000 50  0001 C CNN
+F 0 "#PWR82" H 3500 4000 50  0001 C CNN
 F 1 "GND" H 3500 4100 50  0001 C CNN
 F 2 "" H 3500 4250 50  0000 C CNN
@@
 $EndComp
 $Comp
-L GND #PWR85
+L GND #PWR80
 U 1 1 60FE877B
 P 3100 2600
-F 0 "#PWR85" H 3100 2350 50  0001 C CNN
+F 0 "#PWR80" H 3100 2350 50  0001 C CNN
 F 1 "GND" H 3100 2450 50  0001 C CNN
 F 2 "" H 3100 2600 50  0000 C CNN
@@
 	3100 2600 3200 2600
 Wire Wire Line
-	3650 1150 5500 1150
+	3550 1150 5500 1150
 Wire Wire Line
 	5300 1300 5300 1150
@@
 Wire Wire Line
 	3500 2700 3500 3050
+$Comp
+L L78L06_TO92 U8
+U 1 1 612CE06F
+P 3250 1150
+F 0 "U8" H 3100 1400 50  0000 C CNN
+F 1 "L78L06_TO92" H 3050 1300 50  0000 L CNN
+F 2 "DragonFly:TO-92_Molded_Wide_Oval" H 3250 1375 50  0001 C CIN
+F 3 "" H 3250 1100 50  0001 C CNN
+	1    3250 1150
+	1    0    0    -1
+$EndComp
 $EndSCHEMATC
