File: PCB/KiCAD/IF_SA612_TX.sch (KiCad schematic (older format))
At the start: 19 parts, among them J3 MIC, Q10 MMBT4401LT1G, U8 L78L06_TO92, U9 SA612

Commit message: PCB v1.0
Parts:
- C32, C33, C35, C38: footprint DragonFly:C_0603_HandSoldering -> DragonFly:C_1206_0603
Changed lines of the file:
@@
 $EndDescr
 $Comp
-L GND #PWR82
+L GND #PWR85
 U 1 1 58E1AB18
 P 1750 2050
-F 0 "#PWR82" H 1750 1800 50  0001 C CNN
+F 0 "#PWR85" H 1750 1800 50  0001 C CNN
 F 1 "GND" H 1750 1900 50  0001 C CNN
 F 2 "" H 1750 2050 50  0000 C CNN
@@
 F 0 "C33" H 2300 3850 50  0000 L CNN
 F 1 "100nF" H 2300 3950 50  0000 L CNN
-F 2 "DragonFly:C_0603_HandSoldering" H 2200 3900 50  0001 C CNN
+F 2 "DragonFly:C_1206_0603" H 2200 3900 50  0001 C CNN
 F 3 "" H 2200 3900 50  0000 C CNN
 	1    2200 3900
@@
 $EndComp
 $Comp
-L GND #PWR84
+L GND #PWR87
 U 1 1 58E1AB3A
 P 2950 4000
-F 0 "#PWR84" H 2950 3750 50  0001 C CNN
+F 0 "#PWR87" H 2950 3750 50  0001 C CNN
 F 1 "GND" H 2950 3850 50  0001 C CNN
 F 2 "" H 2950 4000 50  0000 C CNN
@@
 $EndComp
 $Comp
-L GND #PWR83
+L GND #PWR86
 U 1 1 58E1AB40
 P 2200 4000
-F 0 "#PWR83" H 2200 3750 50  0001 C CNN
+F 0 "#PWR86" H 2200 3750 50  0001 C CNN
 F 1 "GND" H 2200 3850 50  0001 C CNN
 F 2 "" H 2200 4000 50  0000 C CNN
@@
 $EndComp
 $Comp
-L GND #PWR86
+L GND #PWR89
 U 1 1 58E1AB6A
 P 3250 1450
-F 0 "#PWR86" H 3250 1200 50  0001 C CNN
+F 0 "#PWR89" H 3250 1200 50  0001 C CNN
 F 1 "GND" H 3250 1300 50  0001 C CNN
 F 2 "" H 3250 1450 50  0000 C CNN
@@
 $EndComp
 $Comp
-L GND #PWR90
+L GND #PWR93
 U 1 1 58E1AB77
 P 5100 2050
-F 0 "#PWR90" H 5100 1800 50  0001 C CNN
+F 0 "#PWR93" H 5100 1800 50  0001 C CNN
 F 1 "GND" H 5100 1900 50  0001 C CNN
 F 2 "" H 5100 2050 50  0000 C CNN
@@
 $EndComp
 $Comp
-L GND #PWR89
+L GND #PWR92
 U 1 1 58E1AB7D
 P 4950 2850
-F 0 "#PWR89" H 4950 2600 50  0001 C CNN
+F 0 "#PWR92" H 4950 2600 50  0001 C CNN
 F 1 "GND" H 4950 2700 50  0001 C CNN
 F 2 "" H 4950 2850 50  0000 C CNN
@@
 F 0 "C38" H 4550 1400 50  0000 L CNN
 F 1 "100nF" H 4550 1500 50  0000 L CNN
-F 2 "DragonFly:C_0603_HandSoldering" H 4800 1400 50  0001 C CNN
+F 2 "DragonFly:C_1206_0603" H 4800 1400 50  0001 C CNN
 F 3 "" H 4800 1400 50  0000 C CNN
 	1    4800 1400
@@
 $EndComp
 $Comp
-L GND #PWR88
+L GND #PWR91
 U 1 1 58E1ABAE
 P 4800 1500
-F 0 "#PWR88" H 4800 1250 50  0001 C CNN
+F 0 "#PWR91" H 4800 1250 50  0001 C CNN
 F 1 "GND" H 4800 1350 50  0001 C CNN
 F 2 "" H 4800 1500 50  0000 C CNN
@@
 $EndComp
 $Comp
-L GND #PWR91
+L GND #PWR94
 U 1 1 58E1ABB4
 P 5300 1500
-F 0 "#PWR91" H 5300 1250 50  0001 C CNN
+F 0 "#PWR94" H 5300 1250 50  0001 C CNN
 F 1 "GND" H 5300 1350 50  0001 C CNN
 F 2 "" H 5300 1500 50  0000 C CNN
@@
 F 0 "C32" H 1850 1950 50  0000 L CNN
 F 1 "100nF" H 1800 2050 50  0000 L CNN
-F 2 "DragonFly:C_0603_HandSoldering" H 1750 1950 50  0001 C CNN
+F 2 "DragonFly:C_1206_0603" H 1750 1950 50  0001 C CNN
 F 3 "" H 1750 1950 50  0000 C CNN
 	1    1750 1950
@@
 Connection ~ 5950 2250
 $Comp
-L GND #PWR92
+L GND #PWR95
 U 1 1 58E1ABEC
 P 5850 2400
-F 0 "#PWR92" H 5850 2150 50  0001 C CNN
+F 0 "#PWR95" H 5850 2150 50  0001 C CNN
 F 1 "GND" H 5850 2250 50  0001 C CNN
 F 2 "" H 5850 2400 50  0000 C CNN
@@
 	5850 2350 6050 2350
 $Comp
-L GND #PWR93
+L GND #PWR96
 U 1 1 58E1ABF4
 P 5850 2950
-F 0 "#PWR93" H 5850 2700 50  0001 C CNN
+F 0 "#PWR96" H 5850 2700 50  0001 C CNN
 F 1 "GND" H 5850 2800 50  0001 C CNN
 F 2 "" H 5850 2950 50  0000 C CNN
@@
 	2950 3800 2950 4000
 $Comp
-L GND #PWR87
+L GND #PWR90
 U 1 1 60FE7FDF
 P 3500 4250
-F 0 "#PWR87" H 3500 4000 50  0001 C CNN
+F 0 "#PWR90" H 3500 4000 50  0001 C CNN
 F 1 "GND" H 3500 4100 50  0001 C CNN
 F 2 "" H 3500 4250 50  0000 C CNN
@@
 F 0 "C35" V 3000 2550 50  0000 L CNN
 F 1 "100nF" V 3150 2550 50  0000 L CNN
-F 2 "DragonFly:C_0603_HandSoldering" H 3300 2600 50  0001 C CNN
+F 2 "DragonFly:C_1206_0603" H 3300 2600 50  0001 C CNN
 F 3 "" H 3300 2600 50  0000 C CNN
 	1    3300 2600
@@
 $EndComp
 $Comp
-L GND #PWR85
+L GND #PWR88
 U 1 1 60FE877B
 P 3100 2600
-F 0 "#PWR85" H 3100 2350 50  0001 C CNN
+F 0 "#PWR88" H 3100 2350 50  0001 C CNN
 F 1 "GND" H 3100 2450 50  0001 C CNN
 F 2 "" H 3100 2600 50  0000 C CNN
