File: PCB/KiCAD/VFO.sch (KiCad schematic (older format))
At the start: 23 parts, among them CON1 AVR-ISP-6, J1 USB_OTG, U10 LD1117S33TR, U2 ATMEGA8-16AU, U3 ADuM1201CR, U6 FT232RL, U7 SI5351, Y7 8Mhz, Y8 27Mhz

Commit message: PCB progress, add digital pin interface, polygon GND, some layout
Parts:
- added J6: Conn_01x10, DragonFly:Pin_Header_Straight_1x10_Pitch2.54mm, symbol Conn_01x10
Connections:
- net +12V: now also J6.10 (Pin_10)
- net +3V3: now also J6.4 (Pin_4)
- net GND: now also J6.3 (Pin_3)
- net SCL: now also J6.2 (Pin_2)
- net SDA: now also J6.1 (Pin_1)
- net IO2: now reaches U2.10 ((AIN0)PD6)
- net IO2: now also J6.6 (Pin_6)
- net IO3: now reaches U2.11 ((AIN1)PD7)
- net IO3: now also J6.7 (Pin_7)
- net IO4: now reaches U2.12 ((ICP)PB0)
- net IO4: now also J6.8 (Pin_8)
- net IO5: now reaches U2.13 ((OC1A)PB1)
- net IO5: now also J6.9 (Pin_9)
- net TX_PA: now reaches U2.14 ((~SS~/OC1B)PB2)
- net IO1: now reaches U2.9 ((T1)PD5)
- net IO1: now also J6.5 (Pin_5)
Other:
- moved on the sheet: C16, C17, U10

Commit message: add FM24CL16,PCB progress
Parts:
- added U14: FM24CL16, DragonFly:SOIC-8_3.9x4.9mm_Pitch1.27mm, symbol FM24CL16
Connections:
- net +3V3: now also U14.8 (VDD)
- net GND: now also U14.4 (VSS)
- net SCL: now also U14.6 (SCL)
- net SDA: now also U14.5 (SDA)
- new net WP: U14.7 (WP)
Changed lines of the file:
@@
 $EndComp
 $Comp
-L GND #PWR017
+L GND #PWR37
 U 1 1 589EB3CB
 P 6100 1350
-F 0 "#PWR017" H 6100 1100 50  0001 C CNN
+F 0 "#PWR37" H 6100 1100 50  0001 C CNN
 F 1 "GND" H 6100 1200 50  0001 C CNN
 F 2 "" H 6100 1350 50  0000 C CNN
@@
 $EndComp
 $Comp
-L GND #PWR018
+L GND #PWR17
 U 1 1 589EFCBC
 P 750 2350
-F 0 "#PWR018" H 750 2100 50  0001 C CNN
+F 0 "#PWR17" H 750 2100 50  0001 C CNN
 F 1 "GND" H 750 2200 50  0001 C CNN
 F 2 "" H 750 2350 50  0000 C CNN
@@
 $EndComp
 $Comp
-L GND #PWR019
+L GND #PWR18
 U 1 1 589EFDB6
 P 750 2800
-F 0 "#PWR019" H 750 2550 50  0001 C CNN
+F 0 "#PWR18" H 750 2550 50  0001 C CNN
 F 1 "GND" H 750 2650 50  0001 C CNN
 F 2 "" H 750 2800 50  0000 C CNN
@@
 $EndComp
 $Comp
-L +3.3V #PWR020
+L +3.3V #PWR38
 U 1 1 58A03CC8
 P 7000 700
-F 0 "#PWR020" H 7000 550 50  0001 C CNN
+F 0 "#PWR38" H 7000 550 50  0001 C CNN
 F 1 "+3.3V" V 7000 1000 50  0000 C CNN
 F 2 "" H 7000 700 50  0000 C CNN
@@
 $EndComp
 $Comp
-L GND #PWR021
+L GND #PWR21
 U 1 1 58A061EE
 P 1300 6150
-F 0 "#PWR021" H 1300 5900 50  0001 C CNN
+F 0 "#PWR21" H 1300 5900 50  0001 C CNN
 F 1 "GND" H 1300 6000 50  0001 C CNN
 F 2 "" H 1300 6150 50  0000 C CNN
@@
 $EndComp
 $Comp
-L GND #PWR022
+L GND #PWR23
 U 1 1 58A09E30
 P 1850 6500
-F 0 "#PWR022" H 1850 6250 50  0001 C CNN
+F 0 "#PWR23" H 1850 6250 50  0001 C CNN
 F 1 "GND" H 1850 6350 50  0001 C CNN
 F 2 "" H 1850 6500 50  0000 C CNN
@@
 $EndComp
 $Comp
-L GND #PWR023
+L GND #PWR25
 U 1 1 58A0C9D9
 P 2600 6500
-F 0 "#PWR023" H 2600 6250 50  0001 C CNN
+F 0 "#PWR25" H 2600 6250 50  0001 C CNN
 F 1 "GND" H 2600 6350 50  0001 C CNN
 F 2 "" H 2600 6500 50  0000 C CNN
@@
 BFO_TX
 $Comp
-L GND #PWR024
+L GND #PWR47
 U 1 1 58E0B7EA
 P 10400 1250
-F 0 "#PWR024" H 10400 1000 50  0001 C CNN
+F 0 "#PWR47" H 10400 1000 50  0001 C CNN
 F 1 "GND" H 10400 1100 50  0001 C CNN
 F 2 "" H 10400 1250 50  0000 C CNN
@@
 SCL
 $Comp
-L +3.3V #PWR025
+L +3.3V #PWR36
 U 1 1 60FBBB98
 P 6100 700
-F 0 "#PWR025" H 6100 550 50  0001 C CNN
+F 0 "#PWR36" H 6100 550 50  0001 C CNN
 F 1 "+3.3V" H 6300 750 50  0000 C CNN
 F 2 "" H 6100 700 50  0000 C CNN
@@
 $EndComp
 $Comp
-L GND #PWR026
+L GND #PWR31
 U 1 1 60FBEFE8
 P 4550 4450
-F 0 "#PWR026" H 4550 4200 50  0001 C CNN
+F 0 "#PWR31" H 4550 4200 50  0001 C CNN
 F 1 "GND" H 4550 4300 50  0001 C CNN
 F 2 "" H 4550 4450 50  0000 C CNN
@@
 $EndComp
 $Comp
-L +3.3V #PWR027
+L +3.3V #PWR30
 U 1 1 60FBF348
 P 4550 3950
-F 0 "#PWR027" H 4550 3800 50  0001 C CNN
+F 0 "#PWR30" H 4550 3800 50  0001 C CNN
 F 1 "+3.3V" V 4550 4200 50  0000 C CNN
 F 2 "" H 4550 3950 50  0000 C CNN
@@
 $EndComp
 $Comp
-L GNDD #PWR028
+L GNDD #PWR43
 U 1 1 60FC3E83
 P 8650 4700
-F 0 "#PWR028" H 8650 4450 50  0001 C CNN
+F 0 "#PWR43" H 8650 4450 50  0001 C CNN
 F 1 "GNDD" H 8650 4575 50  0001 C CNN
 F 2 "" H 8650 4700 50  0001 C CNN
@@
 $EndComp
 $Comp
-L GNDD #PWR029
+L GNDD #PWR42
 U 1 1 60FC3F82
 P 8650 4000
-F 0 "#PWR029" H 8650 3750 50  0001 C CNN
+F 0 "#PWR42" H 8650 3750 50  0001 C CNN
 F 1 "GNDD" H 8650 3875 50  0001 C CNN
 F 2 "" H 8650 4000 50  0001 C CNN
@@
 $EndComp
 $Comp
-L GNDD #PWR030
+L GNDD #PWR46
 U 1 1 60FC3FE1
 P 10250 4750
-F 0 "#PWR030" H 10250 4500 50  0001 C CNN
+F 0 "#PWR46" H 10250 4500 50  0001 C CNN
 F 1 "GNDD" H 10250 4625 50  0001 C CNN
 F 2 "" H 10250 4750 50  0001 C CNN
@@
 $EndComp
 $Comp
-L GNDD #PWR031
+L GNDD #PWR35
 U 1 1 60FC45C5
 P 5650 4450
-F 0 "#PWR031" H 5650 4200 50  0001 C CNN
+F 0 "#PWR35" H 5650 4200 50  0001 C CNN
 F 1 "GNDD" H 5650 4325 50  0001 C CNN
 F 2 "" H 5650 4450 50  0001 C CNN
@@
 $EndComp
 $Comp
-L GNDD #PWR032
+L GNDD #PWR39
 U 1 1 60FC465C
 P 7000 5900
-F 0 "#PWR032" H 7000 5650 50  0001 C CNN
+F 0 "#PWR39" H 7000 5650 50  0001 C CNN
 F 1 "GNDD" H 7000 5775 50  0001 C CNN
 F 2 "" H 7000 5900 50  0001 C CNN
@@
 $EndComp
 $Comp
-L GNDD #PWR033
+L GNDD #PWR44
 U 1 1 60FC82A8
 P 8700 3600
-F 0 "#PWR033" H 8700 3350 50  0001 C CNN
+F 0 "#PWR44" H 8700 3350 50  0001 C CNN
 F 1 "GNDD" H 8700 3475 50  0001 C CNN
 F 2 "" H 8700 3600 50  0001 C CNN
@@
 $EndComp
 $Comp
-L GNDD #PWR034
+L GNDD #PWR45
 U 1 1 60FC8353
 P 9650 3600
-F 0 "#PWR034" H 9650 3350 50  0001 C CNN
+F 0 "#PWR45" H 9650 3350 50  0001 C CNN
 F 1 "GNDD" H 9650 3475 50  0001 C CNN
 F 2 "" H 9650 3600 50  0001 C CNN
@@
 $EndComp
 $Comp
-L GNDD #PWR035
+L GNDD #PWR41
 U 1 1 60FC83BE
 P 7600 3550
-F 0 "#PWR035" H 7600 3300 50  0001 C CNN
+F 0 "#PWR41" H 7600 3300 50  0001 C CNN
 F 1 "GNDD" H 7600 3425 50  0001 C CNN
 F 2 "" H 7600 3550 50  0001 C CNN
@@
 $EndComp
 $Comp
-L +3.3V #PWR036
+L +3.3V #PWR26
 U 1 1 60FCB4EA
 P 2650 1250
-F 0 "#PWR036" H 2650 1100 50  0001 C CNN
+F 0 "#PWR26" H 2650 1100 50  0001 C CNN
 F 1 "+3.3V" H 2850 1300 50  0000 C CNN
 F 2 "" H 2650 1250 50  0000 C CNN
@@
 	4950 1450 1600 1450
 $Comp
-L GND #PWR037
+L GND #PWR24
 U 1 1 60FCC081
 P 2600 4550
-F 0 "#PWR037" H 2600 4300 50  0001 C CNN
+F 0 "#PWR24" H 2600 4300 50  0001 C CNN
 F 1 "GND" H 2600 4400 50  0001 C CNN
 F 2 "" H 2600 4550 50  0000 C CNN
@@
 Connection ~ 2600 4500
 $Comp
-L +3.3V #PWR038
+L +3.3V #PWR27
 U 1 1 60FCC6C5
 P 3150 5850
-F 0 "#PWR038" H 3150 5700 50  0001 C CNN
+F 0 "#PWR27" H 3150 5700 50  0001 C CNN
 F 1 "+3.3V" V 3150 6100 50  0000 C CNN
 F 2 "" H 3150 5850 50  0000 C CNN
@@
 $EndComp
 $Comp
-L +12V #PWR039
+L +12V #PWR19
 U 1 1 60FCCDC8
 P 750 5750
-F 0 "#PWR039" H 750 5600 50  0001 C CNN
+F 0 "#PWR19" H 750 5600 50  0001 C CNN
 F 1 "+12V" H 750 5890 50  0000 C CNN
 F 2 "" H 750 5750 50  0000 C CNN
@@
 TX_TRX
 $Comp
-L GND #PWR040
+L GND #PWR22
 U 1 1 60FE3270
 P 1650 2200
-F 0 "#PWR040" H 1650 1950 50  0001 C CNN
+F 0 "#PWR22" H 1650 1950 50  0001 C CNN
 F 1 "GND" H 1650 2050 50  0001 C CNN
 F 2 "" H 1650 2200 50  0000 C CNN
@@
 $EndComp
 $Comp
-L GND #PWR041
+L GND #PWR20
 U 1 1 610504BE
 P 1150 2100
-F 0 "#PWR041" H 1150 1850 50  0001 C CNN
+F 0 "#PWR20" H 1150 1850 50  0001 C CNN
 F 1 "GND" H 1150 1950 50  0001 C CNN
 F 2 "" H 1150 2100 50  0000 C CNN
@@
 $EndComp
 $Comp
-L GND #PWR042
+L GND #PWR40
 U 1 1 61063FC6
 P 7100 1100
-F 0 "#PWR042" H 7100 850 50  0001 C CNN
+F 0 "#PWR40" H 7100 850 50  0001 C CNN
 F 1 "GND" H 7100 950 50  0001 C CNN
 F 2 "" H 7100 1100 50  0000 C CNN
@@
 	5100 5750 5650 5750
 $Comp
-L GND #PWR043
+L GND #PWR34
 U 1 1 612677D4
 P 5450 5850
-F 0 "#PWR043" H 5450 5600 50  0001 C CNN
+F 0 "#PWR34" H 5450 5600 50  0001 C CNN
 F 1 "GND" H 5450 5700 50  0001 C CNN
 F 2 "" H 5450 5850 50  0000 C CNN
@@
 	5450 5850 5650 5850
 $Comp
-L +3.3V #PWR044
+L +3.3V #PWR32
 U 1 1 61267C9A
 P 5100 5950
-F 0 "#PWR044" H 5100 5800 50  0001 C CNN
+F 0 "#PWR32" H 5100 5800 50  0001 C CNN
 F 1 "+3.3V" V 5100 6200 50  0000 C CNN
 F 2 "" H 5100 5950 50  0000 C CNN
@@
 	5450 6450 5650 6450
 $Comp
-L +12V #PWR045
+L +12V #PWR33
 U 1 1 6126AF05
 P 5100 6550
-F 0 "#PWR045" H 5100 6400 50  0001 C CNN
+F 0 "#PWR33" H 5100 6400 50  0001 C CNN
 F 1 "+12V" V 5100 6800 50  0000 C CNN
 F 2 "" H 5100 6550 50  0000 C CNN
@@
 Text GLabel 4850 2000 2    60   Output ~ 0
 TX_PA
+Wire Wire Line
+	4250 6900 4500 6900
+Wire Wire Line
+	4250 7050 4500 7050
+$Comp
+L +3.3V #PWR28
+U 1 1 612F3450
+P 3850 6550
+F 0 "#PWR28" H 3850 6400 50  0001 C CNN
+F 1 "+3.3V" V 3850 6800 50  0000 C CNN
+F 2 "" H 3850 6550 50  0000 C CNN
+F 3 "" H 3850 6550 50  0000 C CNN
+	1    3850 6550
+	1    0    0    -1
+$EndComp
+Wire Wire Line
+	3850 6550 3850 6650
+Text GLabel 4500 7050 2    60   Input ~ 0
+SCL
+Text GLabel 4500 6900 2    60   Input ~ 0
+SDA
+$Comp
+L FM24CL16 U14
+U 1 1 612F3845
+P 3850 7000
+F 0 "U14" H 3650 7250 50  0000 C CNN
+F 1 "FM24CL16" H 4100 6700 50  0000 C CNN
+F 2 "DragonFly:SOIC-8_3.9x4.9mm_Pitch1.27mm" H 3850 7000 50  0001 C CNN
+F 3 "" H 3850 7000 50  0001 C CNN
+	1    3850 7000
+	1    0    0    -1
+$EndComp
+$Comp
+L GND #PWR29
+U 1 1 612F38B9
+P 3850 7400
+F 0 "#PWR29" H 3850 7150 50  0001 C CNN
+F 1 "GND" H 3850 7250 50  0001 C CNN
+F 2 "" H 3850 7400 50  0000 C CNN
+F 3 "" H 3850 7400 50  0000 C CNN
+	1    3850 7400
+	1    0    0    -1
+$EndComp
+Wire Wire Line
+	3450 7200 3250 7200
+Text GLabel 3250 7200 0    60   Input ~ 0
+WP
 $EndSCHEMATC

Commit message: PCB v1.0
Parts:
- added C79, C80: 100nF, DragonFly:C_1206_0603, symbol C_Small
- added R44, R45, R46, R47, R48: 56R, DragonFly:R_0603_HandSoldering, symbol R_Small
- C16, C37, C54: footprint Capacitors_SMD:C_0603_HandSoldering -> DragonFly:C_1206_0603
- R6, R7: footprint Resistors_SMD:R_0603_HandSoldering -> DragonFly:R_1206_0603
Connections:
- net +3V3: now also C79.2, C80.1
- net GND: now also C79.1, C80.2
- net IO1: now also R44.1; no longer J6.5 (Pin_5)
- net IO2: now also R45.1; no longer J6.6 (Pin_6)
- net IO3: now also R46.1; no longer J6.7 (Pin_7)
- net IO4: now also R47.1; no longer J6.8 (Pin_8)
- net IO5: now also R48.1; no longer J6.9 (Pin_9)
- net WP: now also U2.26 ((ADC3)PC3)
- net AGC_OFF: now reaches U2.25 ((ADC2)PC2)
- new net: J6.5 (Pin_5), R44.2
- new net: J6.6 (Pin_6), R45.2
- new net: J6.7 (Pin_7), R46.2
- new net: J6.8 (Pin_8), R47.2
- new net: J6.9 (Pin_9), R48.2
Other:
- moved on the sheet: C16, C17, U10, U14
